File: KiCad/TestPCB/TestPCB.kicad_pcb (KiCad board)
At the start: 2 copper layers, 102.1 x 148.4 mm, 92 parts, among them J1 Conn_01x01_Male, J2 Conn_01x01_Male, U1 MC33078, U10a1 OP07, U10b1 OP07, U11a1 OP07, U11b1 OP07, U12a1 OP07, U12b1 OP07, U2 MC33078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

Commit message: Fixing PCB design
Parts:
- added JPin_U13b1: Jumper_2_Bridged, Connector_PinHeader_2.54mm:PinHeader_1x02_P2.54mm_Vertical, F.Cu at (51.3, 146.2)
- added JPin_U1a1: Jumper_2_Bridged, Connector_PinHeader_2.54mm:PinHeader_1x02_P2.54mm_Vertical, F.Cu at (53.8, 28.7)
- added JPin_U1b1: Jumper_2_Bridged, Connector_PinHeader_2.54mm:PinHeader_1x02_P2.54mm_Vertical, F.Cu at (53.7, 35.1)
- added JPin_U2a1: Jumper_2_Bridged, Connector_PinHeader_2.54mm:PinHeader_1x02_P2.54mm_Vertical, F.Cu at (54.3, 53.4)
- added JPin_U2b1: Jumper_2_Bridged, Connector_PinHeader_2.54mm:PinHeader_1x02_P2.54mm_Vertical, F.Cu at (54.1, 60.1)
- added JPin_U3a1: Jumper_2_Bridged, Connector_PinHeader_2.54mm:PinHeader_1x02_P2.54mm_Vertical, F.Cu at (51.3, 138.9)
- added JPin_U4a1: Jumper_2_Bridged, Connector_PinHeader_2.54mm:PinHeader_1x02_P2.54mm_Vertical, F.Cu at (52.4, 91.2)
- added JPin_U4b1: Jumper_2_Bridged, Connector_PinHeader_2.54mm:PinHeader_1x02_P2.54mm_Vertical, F.Cu at (52.4, 97.8)
- J1, J2, Jout10a1, Jout10b1, Jout11a1, Jout11b1, Jout12a1, Jout12b1, Jout5, Jout6, Jout7, Jout8, Jout9a1, Jout9b1: footprint Connector_PinHeader_2.00mm:PinHeader_1x01_P2.00mm_Vertical -> Connector_PinHeader_2.54mm:PinHeader_1x01_P2.54mm_Vertical
- JPout_U1a1, JPout_U1b1, JPout_U2a1, JPout_U2b1, JPout_U3a1, JPout_U3b1, JPout_U4a1, JPout_U4b1: footprint Connector_PinHeader_2.00mm:PinHeader_1x02_P2.00mm_Vertical -> Connector_PinHeader_2.54mm:PinHeader_1x02_P2.54mm_Vertical
- J_LDAC_SYNC_SCL_SDA1: footprint Connector_PinHeader_2.00mm:PinHeader_1x04_P2.00mm_Vertical -> Connector_PinHeader_2.54mm:PinHeader_1x04_P2.54mm_Vertical
- moved TP_U1a1 6.07 mm to (48.5, 30.0)
- moved TP_U1b1 6.06 mm to (48.5, 36.5)
- moved TP_U2a1 5.77 mm to (48.7, 54.4)
- moved TP_U2b1 5.60 mm to (48.8, 61.2)
- moved TP_U3a1 4.19 mm to (45.9, 139.9)
- moved TP_U3b1 4.19 mm to (45.9, 146.8)
- moved TP_U4a1 3.54 mm to (47.3, 91.9)
- moved TP_U4b1 3.54 mm to (47.3, 98.2)
Connections:
- J_LDAC_SYNC_SCL_SDA1 pad 2: +5V -> Net-(J_LDAC_SYNC_SCL_SDA1-Pad2)
- TP_U1a1 pad 1: Net-(TP_U1a1-Pad1) -> Net-(Udac1-Pad13)
- TP_U1b1 pad 1: Net-(TP_U1b1-Pad1) -> Net-(Udac1-Pad12)
- TP_U2a1 pad 1: Net-(TP_U2a1-Pad1) -> Net-(Udac1-Pad11)
- TP_U2b1 pad 1: +2V5 -> Net-(Udac1-Pad10)
- TP_U3b1 pad 1: +5V -> Net-(TP_U3b1-Pad1)
- TP_U4a1 pad 1: +2V5 -> Net-(Udac1-Pad7)
- TP_U4b1 pad 1: Net-(TP_U4b1-Pad1) -> Net-(Udac1-Pad6)
- U1 pad 3: Net-(TP_U1a1-Pad1) -> Net-(U1-Pad3)
- U1 pad 5: Net-(TP_U1b1-Pad1) -> Net-(U1-Pad5)
- U2 pad 3: Net-(TP_U2a1-Pad1) -> Net-(U2-Pad3)
- U2 pad 5: +2V5 -> Net-(U2-Pad5)
- U3 pad 3: Net-(TP_U3a1-Pad1) -> Net-(U3-Pad3)
- U3 pad 5: +5V -> Net-(U3-Pad5)
- U4 pad 3: +2V5 -> Net-(U4-Pad3)
- U4 pad 5: Net-(TP_U4b1-Pad1) -> Net-(U4-Pad5)
- Udac1 pad 10: +2V5 -> Net-(Udac1-Pad10)
- Udac1 pad 11: Net-(TP_U2a1-Pad1) -> Net-(Udac1-Pad11)
- Udac1 pad 12: Net-(TP_U1b1-Pad1) -> Net-(Udac1-Pad12)
- Udac1 pad 13: Net-(TP_U1a1-Pad1) -> Net-(Udac1-Pad13)
- Udac1 pad 2: +5V -> Net-(J_LDAC_SYNC_SCL_SDA1-Pad2)
- Udac1 pad 4: +5V -> Net-(TP_U3b1-Pad1)
- Udac1 pad 6: Net-(TP_U4b1-Pad1) -> Net-(Udac1-Pad6)
- Udac1 pad 7: +2V5 -> Net-(Udac1-Pad7)
Routing:
- net +5V: track 627.7 -> 506.1 mm
- net +2V5: track 291.2 -> 179.9 mm
- net Net-(TP_U1b1-Pad1): track 88.7 -> 0.00 mm
- net Net-(TP_U1a1-Pad1): track 86.1 -> 0.00 mm
- net Net-(TP_U3b1-Pad1): track 0.00 -> 85.1 mm
- net Net-(Udac1-Pad13): track 0.00 -> 69.3 mm
- net Net-(Udac1-Pad12): track 0.00 -> 65.1 mm
- net Net-(TP_U2a1-Pad1): track 63.1 -> 0.00 mm
- net Net-(TP_U4b1-Pad1): track 61.0 -> 0.00 mm
- net Net-(Udac1-Pad11): track 0.00 -> 46.1 mm
- net Net-(Udac1-Pad10): track 0.00 -> 40.1 mm
- net Net-(Udac1-Pad6): track 0.00 -> 35.1 mm
- net Net-(Udac1-Pad7): track 0.00 -> 32.8 mm
- net Net-(U1-Pad5): track 0.00 -> 28.5 mm
- net Net-(U2-Pad5): track 0.00 -> 28.4 mm
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