File: KiCad/TestPCB/TestPCB.kicad_pcb (KiCad board)
At the start: 2 copper layers, 91 parts, among them U1 MC33078, U10a1 OP07, U10b1 OP07, U11a1 OP07, U11b1 OP07, U12a1 OP07, U12b1 OP07, U2 MC33078, U3 MC33078, U4 MC33078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

Commit message: PCB update
Parts:
- moved J_SYNC1 165.1 mm to (27.9, 109.2)
- moved TPRef1 153.0 mm to (35.6, 63.5)
- moved J_SCL1 146.5 mm to (27.9, 94.0)
- moved J_SDA1 140.5 mm to (27.9, 99.1)
- moved J_LDAC1 138.4 mm to (27.9, 104.1)
- moved TP_U4a1 123.6 mm to (66.0, 147.3)
- moved Udac1 116.5 mm to (38.1, 88.9), turned to 90 degrees
- moved TP_U2b1 115.5 mm to (63.5, 73.7)
- moved TP_U1a1 112.3 mm to (61.0, 38.7)
- moved TP_U4b1 109.7 mm to (66.0, 154.9)
- moved TP_U3a1 108.1 mm to (63.5, 109.2)
- moved TP_U1b1 105.9 mm to (61.0, 45.1)
- moved R_SCL1 101.8 mm to (22.9, 83.8)
- moved U9 100.5 mm to (27.9, 68.6)
- moved Cref1 91.6 mm to (20.3, 66.0), turned to -90 degrees
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Routing:
- net Net-(Rain_U5-Pad2): track 0.00 -> 12.6 mm
- net Net-(Rain_U6-Pad2): track 0.00 -> 12.2 mm
- net GND: track 0.00 -> 12.1 mm
- net Net-(U6-Pad2): track 0.00 -> 10.6 mm
- net Net-(U5-Pad2): track 0.00 -> 10.6 mm
- net Net-(JPout_U1a1-Pad2): track 0.00 -> 6.97 mm
- net Net-(JPout_U1b1-Pad2): track 0.00 -> 6.19 mm

Commit message: PCB progress, our outputs done
Parts:
- TPRef1: value TestPoint -> Conn_01x01_Male; footprint TestPoint:TestPoint_Pad_4.0x4.0mm -> Connector_PinHeader_2.54mm:PinHeader_1x01_P2.54mm_Vertical
- U10a1, U10b1, U11a1, U11b1, U12a1, U12b1, U5, U6, U7, U8, U9a1, U9b1: footprint Package_SO:SOIC-8_3.9x4.9mm_P1.27mm -> Package_DIP:DIP-8_W7.62mm_Socket_LongPads
- moved JPout_U3a1 113.5 mm to (232.8, 100.7)
- moved JPout_U3b1 113.5 mm to (232.8, 110.8)
- moved JPout_U4a1 113.5 mm to (232.8, 138.8)
- moved JPout_U4b1 113.5 mm to (232.8, 151.5)
- moved Jout10a1 113.5 mm to (273.5, 110.8)
- moved Jout10b1 113.5 mm to (273.5, 118.4)
- moved Jout9a1 113.5 mm to (273.5, 95.6)
- moved Jout9b1 113.5 mm to (273.5, 103.2)
- moved Rain_U9 113.5 mm to (243.0, 95.6)
- moved Rbin_U12 113.5 mm to (245.4, 154.0)
- moved Rcin_U12 113.5 mm to (245.4, 159.1)
- moved Rf_U3a1 113.5 mm to (204.9, 108.3)
- moved Rf_U3b1 113.5 mm to (204.9, 118.4)
- moved Rf_U4a1 113.5 mm to (204.9, 146.4)
- moved Rf_U4b1 113.5 mm to (204.9, 156.5)
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Connections:
- net Net-(Rin-_U1a1-Pad1) renamed +2V5
- TP_U1a1 pad 1: Net-(TP_U1a1-Pad1) -> Net-(Udac1-Pad13)
- TP_U2b1 pad 1: Net-(TP_U2b1-Pad1) -> Net-(Udac1-Pad10)
- TP_U3b1 pad 1: Net-(Udac1-Pad11) -> Net-(TP_U3b1-Pad1)
- TP_U4a1 pad 1: Net-(Udac1-Pad7) -> Net-(TP_U4a1-Pad1)
- TP_U4b1 pad 1: Net-(Udac1-Pad10) -> Net-(TP_U4b1-Pad1)
- U1 pad 3: Net-(TP_U1a1-Pad1) -> Net-(Udac1-Pad13)
- U2 pad 5: Net-(TP_U2b1-Pad1) -> Net-(Udac1-Pad10)
- U3 pad 5: Net-(Udac1-Pad11) -> Net-(TP_U3b1-Pad1)
- U4 pad 3: Net-(Udac1-Pad7) -> Net-(TP_U4a1-Pad1)
- U4 pad 5: Net-(Udac1-Pad10) -> Net-(TP_U4b1-Pad1)
- Udac1 pad 11: Net-(Udac1-Pad11) -> Net-(TP_U2a1-Pad1)
- Udac1 pad 12: Net-(TP_U2b1-Pad1) -> Net-(TP_U1b1-Pad1)
- Udac1 pad 13: Net-(TP_U1b1-Pad1) -> Net-(Udac1-Pad13)
- Udac1 pad 4: Net-(TP_U1a1-Pad1) -> Net-(TP_U3a1-Pad1)
- Udac1 pad 5: Net-(TP_U2a1-Pad1) -> Net-(TP_U3b1-Pad1)
- Udac1 pad 6: Net-(TP_U3a1-Pad1) -> Net-(TP_U4a1-Pad1)
- Udac1 pad 7: Net-(Udac1-Pad7) -> Net-(TP_U4b1-Pad1)
Routing:
- net +5V: track 0.00 -> 145.3 mm
- net -5V: track 0.00 -> 135.2 mm
- net +2V5: track 0.00 -> 63.1 mm
- net GND: track 12.1 -> 42.5 mm
- net Net-(Udac1-Pad10): track 0.00 -> 28.3 mm
- net Net-(TP_U1b1-Pad1): track 0.00 -> 28.0 mm
- net Net-(TP_U3a1-Pad1): track 0.00 -> 23.8 mm
- net Net-(JPout_U1a1-Pad1): track 0.00 -> 23.5 mm
- net Net-(JPout_U2a1-Pad1): track 0.00 -> 23.4 mm
- net Net-(Rf_U2b1-Pad1): track 0.00 -> 21.8 mm
- net Net-(TP_U3b1-Pad1): track 0.00 -> 21.4 mm
- net Net-(Rf_U1b1-Pad1): track 0.00 -> 20.9 mm
- net Net-(TP_U2a1-Pad1): track 0.00 -> 19.7 mm
- net Net-(J_SCL1-Pad1): track 0.00 -> 19.6 mm
- net Net-(Udac1-Pad13): track 0.00 -> 19.3 mm
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
Commit message: First PCB run done
Parts:
- moved U11a1 165.9 mm to (108.8, 71.3)
- moved Jout11a1 164.9 mm to (121.4, 76.3)
- moved U11b1 164.3 mm to (108.7, 83.3)
- moved Jout11b1 163.5 mm to (121.3, 88.2)
- moved U12a1 162.9 mm to (108.6, 95.5)
- moved U12b1 162.5 mm to (108.5, 107.1)
- moved Jout12a1 162.2 mm to (121.3, 100.4)
- moved Jout12b1 161.2 mm to (121.1, 112.1)
- moved Rain_U12 160.7 mm to (93.5, 96.8), turned to 90 degrees
- moved U10b1 159.6 mm to (108.2, 155.8)
- moved Rin-_U4b1 159.1 mm to (55.6, 96.4)
- moved Rain_U11 158.5 mm to (93.4, 89.3), turned to -90 degrees
- moved U10a1 158.5 mm to (108.3, 143.7)
- moved Jout10b1 158.2 mm to (121.0, 160.9)
- moved Rbin_U12 157.5 mm to (98.6, 97.1), turned to 90 degrees
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Connections:
- TP_U4a1 pad 1: Net-(TP_U4a1-Pad1) -> Net-(Udac1-Pad7)
- TP_U4b1 pad 1: Net-(TP_U4b1-Pad1) -> Net-(Udac1-Pad6)
- U4 pad 3: Net-(TP_U4a1-Pad1) -> Net-(Udac1-Pad7)
- U4 pad 5: Net-(TP_U4b1-Pad1) -> Net-(Udac1-Pad6)
- Udac1 pad 4: Net-(TP_U3a1-Pad1) -> Net-(TP_U3b1-Pad1)
- Udac1 pad 5: Net-(TP_U3b1-Pad1) -> Net-(TP_U3a1-Pad1)
- Udac1 pad 6: Net-(TP_U4a1-Pad1) -> Net-(Udac1-Pad6)
- Udac1 pad 7: Net-(TP_U4b1-Pad1) -> Net-(Udac1-Pad7)
Routing:
- net +5V: track 145.3 -> 480.5 mm
- net -5V: track 135.2 -> 389.6 mm
- net +2V5: track 63.1 -> 176.8 mm
- net Net-(TP_U3b1-Pad1): track 21.4 -> 108.3 mm
- net Net-(TP_U3a1-Pad1): track 23.8 -> 90.7 mm
- net Net-(Udac1-Pad13): track 19.3 -> 86.1 mm
- net Net-(Udac1-Pad6): track 0.00 -> 61.0 mm
- net Net-(TP_U1b1-Pad1): track 28.0 -> 88.7 mm
- net Net-(Udac1-Pad7): track 0.00 -> 49.1 mm
- net Net-(TP_U2a1-Pad1): track 19.7 -> 63.1 mm
- net Net-(Udac1-Pad10): track 28.3 -> 64.6 mm
- net Net-(Rain_U9-Pad2): track 0.00 -> 23.4 mm
- net Net-(JPout_U3a1-Pad1): track 0.00 -> 23.2 mm
- net Net-(Rain_U11-Pad2): track 0.00 -> 22.8 mm
- net Net-(JPout_U4a1-Pad1): track 0.00 -> 22.3 mm
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- added copper zone on B.Cu, net GND

Commit message: Added GND pins
Parts:
- added J1: Conn_01x01_Male, Connector_PinHeader_2.54mm:PinHeader_1x01_P2.54mm_Vertical, F.Cu at (28.5, 30.4)
- added J2: Conn_01x01_Male, Connector_PinHeader_2.54mm:PinHeader_1x01_P2.54mm_Vertical, F.Cu at (31.3, 147.1)
Changed lines of the file:
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@@
+    )
+  )
+  (footprint "Connector_PinHeader_2.54mm:PinHeader_1x01_P2.54mm_Vertical" (layer "F.Cu")
+    (at 31.27 147.05)
+    (descr "Through hole straight pin header, 1x01, 2.54mm pitch, single row")
+    (tags "Through hole pin header THT 1x01 2.54mm single row")
+    (property "Sheetfile" "TestPCB.kicad_sch")
+    (property "Sheetname" "")
+    (attr through_hole)
+    (fp_text reference "J2" (at 0 -2.33) (layer "F.SilkS")
+      (effects (font (size 1 1) (thickness 0.15)))
+    )
+    (fp_text value "Conn_01x01_Male" (at 0 2.33) (layer "F.Fab")
+      (effects (font (size 1 1) (thickness 0.15)))
+    )
+    (fp_text user "${REFERENCE}" (at 0 0 90) (layer "F.Fab")
+      (effects (font (size 1 1) (thickness 0.15)))
+    )
+    (fp_line (start -1.33 1.27) (end -1.33 1.33) (layer "F.SilkS") (width 0.12))
+    (fp_line (start -1.33 1.27) (end 1.33 1.27) (layer "F.SilkS") (width 0.12))
+    (fp_line (start -1.33 0) (end -1.33 -1.33) (layer "F.SilkS") (width 0.12))
+    (fp_line (start 1.33 1.27) (end 1.33 1.33) (layer "F.SilkS") (width 0.12))
+    (fp_line (start -1.33 -1.33) (end 0 -1.33) (layer "F.SilkS") (width 0.12))
+    (fp_line (start -1.33 1.33) (end 1.33 1.33) (layer "F.SilkS") (width 0.12))
+    (fp_line (start -1.8 -1.8) (end -1.8 1.8) (layer "F.CrtYd") (width 0.05))
+    (fp_line (start -1.8 1.8) (end 1.8 1.8) (layer "F.CrtYd") (width 0.05))
+    (fp_line (start 1.8 1.8) (end 1.8 -1.8) (layer "F.CrtYd") (width 0.05))
+    (fp_line (start 1.8 -1.8) (end -1.8 -1.8) (layer "F.CrtYd") (width 0.05))
+    (fp_line (start -1.27 -0.635) (end -0.635 -1.27) (layer "F.Fab") (width 0.1))
+    (fp_line (start -0.635 -1.27) (end 1.27 -1.27) (layer "F.Fab") (width 0.1))
+    (fp_line (start 1.27 1.27) (end -1.27 1.27) (layer "F.Fab") (width 0.1))
+    (fp_line (start 1.27 -1.27) (end 1.27 1.27) (layer "F.Fab") (width 0.1))
+    (fp_line (start -1.27 1.27) (end -1.27 -0.635) (layer "F.Fab") (width 0.1))
+    (pad "1" thru_hole rect (at 0 0) (size 1.7 1.7) (drill 1) (layers *.Cu *.Mask)
+      (net 1 "GND") (pinfunction "Pin_1") (pintype "passive"))
+    (model "${KICAD6_3DMODEL_DIR}/Connector_PinHeader_2.54mm.3dshapes/PinHeader_1x01_P2.54mm_Vertical.wrl"
+      (offset (xyz 0 0 0))
+      (scale (xyz 1 1 1))
+      (rotate (xyz 0 0 0))
     )
   )
@@
       (offset (xyz 0 0 0))
       (scale (xyz 1 1 1))
+      (rotate (xyz 0 0 0))
+    )
+  )
+  (footprint "Connector_PinHeader_2.54mm:PinHeader_1x01_P2.54mm_Vertical" (layer "F.Cu")
+    (at 28.51 30.43)
+    (descr "Through hole straight pin header, 1x01, 2.54mm pitch, single row")
+    (tags "Through hole pin header THT 1x01 2.54mm single row")
+    (property "Sheetfile" "TestPCB.kicad_sch")
+    (property "Sheetname" "")
+    (attr through_hole)
+    (fp_text reference "J1" (at 0 -2.33) (layer "F.SilkS")
+      (effects (font (size 1 1) (thickness 0.15)))
+    )
+    (fp_text value "Conn_01x01_Male" (at 0 2.33) (layer "F.Fab")
+      (effects (font (size 1 1) (thickness 0.15)))
+    )
+    (fp_text user "${REFERENCE}" (at 0 0 90) (layer "F.Fab")
+      (effects (font (size 1 1) (thickness 0.15)))
+    )
+    (fp_line (start -1.33 1.27) (end 1.33 1.27) (layer "F.SilkS") (width 0.12))
+    (fp_line (start 1.33 1.27) (end 1.33 1.33) (layer "F.SilkS") (width 0.12))
+    (fp_line (start -1.33 1.27) (end -1.33 1.33) (layer "F.SilkS") (width 0.12))
+    (fp_line (start -1.33 -1.33) (end 0 -1.33) (layer "F.SilkS") (width 0.12))
+    (fp_line (start -1.33 1.33) (end 1.33 1.33) (layer "F.SilkS") (width 0.12))
+    (fp_line (start -1.33 0) (end -1.33 -1.33) (layer "F.SilkS") (width 0.12))
+    (fp_line (start -1.8 -1.8) (end -1.8 1.8) (layer "F.CrtYd") (width 0.05))
+    (fp_line (start 1.8 -1.8) (end -1.8 -1.8) (layer "F.CrtYd") (width 0.05))
+    (fp_line (start -1.8 1.8) (end 1.8 1.8) (layer "F.CrtYd") (width 0.05))
+    (fp_line (start 1.8 1.8) (end 1.8 -1.8) (layer "F.CrtYd") (width 0.05))
+    (fp_line (start -1.27 -0.635) (end -0.635 -1.27) (layer "F.Fab") (width 0.1))
+    (fp_line (start -1.27 1.27) (end -1.27 -0.635) (layer "F.Fab") (width 0.1))
+    (fp_line (start 1.27 1.27) (end -1.27 1.27) (layer "F.Fab") (width 0.1))
+    (fp_line (start -0.635 -1.27) (end 1.27 -1.27) (layer "F.Fab") (width 0.1))
+    (fp_line (start 1.27 -1.27) (end 1.27 1.27) (layer "F.Fab") (width 0.1))
+    (pad "1" thru_hole rect (at 0 0) (size 1.7 1.7) (drill 1) (layers *.Cu *.Mask)
+      (net 1 "GND") (pinfunction "Pin_1") (pintype "passive"))
+    (model "${KICAD6_3DMODEL_DIR}/Connector_PinHeader_2.54mm.3dshapes/PinHeader_1x01_P2.54mm_Vertical.wrl"
+      (offset (xyz 0 0 0))
+      (scale (xyz 1 1 1))

Commit message: finished desing
Parts:
- removed J_LDAC1, J_SCL1, J_SDA1, J_SYNC1: Conn_01x01_Male, Connector_PinHeader_2.54mm:PinHeader_1x01_P2.54mm_Vertical
- added J_LDAC_SYNC_SCL_SDA1: Conn_01x04_Male, Connector_PinHeader_2.00mm:PinHeader_1x04_P2.00mm_Vertical, F.Cu at (24.7, 74.7)
- added TPRef2: Conn_01x01_Male, Connector_PinHeader_2.54mm:PinHeader_1x01_P2.54mm_Vertical, F.Cu at (98.4, 164.0)
- added TPRef3: Conn_01x01_Male, Connector_PinHeader_2.54mm:PinHeader_1x01_P2.54mm_Vertical, F.Cu at (86.3, 163.7)
- Cref1: footprint Capacitor_THT:C_Disc_D5.0mm_W2.5mm_P5.00mm -> Capacitor_THT:C_Disc_D5.0mm_W2.5mm_P2.50mm
- J1, J2, Jout10a1, Jout10b1, Jout11a1, Jout11b1, Jout12a1, Jout12b1, Jout5, Jout6, Jout7, Jout8, Jout9a1, Jout9b1: footprint Connector_PinHeader_2.54mm:PinHeader_1x01_P2.54mm_Vertical -> Connector_PinHeader_2.00mm:PinHeader_1x01_P2.00mm_Vertical
- JPout_U1a1, JPout_U1b1, JPout_U2a1, JPout_U2b1, JPout_U3a1, JPout_U3b1, JPout_U4a1, JPout_U4b1: footprint Connector_PinHeader_2.54mm:PinHeader_1x02_P2.54mm_Vertical -> Connector_PinHeader_2.00mm:PinHeader_1x02_P2.00mm_Vertical
- Rain_U10, Rain_U11, Rain_U12, Rain_U5, Rain_U6, Rain_U7, Rain_U8, Rain_U9, Rbin_U10, Rbin_U11, Rbin_U12, Rbin_U5, Rbin_U6, Rbin_U7, Rbin_U8, Rbin_U9, Rcin_U10, Rcin_U11, Rcin_U12, Rcin_U9: footprint Resistor_SMD:R_2010_5025Metric_Pad1.40x2.65mm_HandSolder -> Resistor_SMD:R_1206_3216Metric_Pad1.30x1.75mm_HandSolder
- moved J2 46.3 mm to (74.4, 163.9)
Routing:
- net +5V: track 480.5 -> 506.1 mm
- net -5V: track 389.6 -> 404.8 mm
- net Net-(Udac1-Pad2): track 6.82 -> 12.1 mm
- net Net-(Udac1-Pad1): track 8.30 -> 12.7 mm
- net GND: track 59.3 -> 61.3 mm
- net Net-(Rain_U5-Pad2): track 10.9 -> 9.28 mm
- net Net-(JPout_U3b1-Pad2): track 5.77 -> 4.44 mm
- net Net-(Rain_U12-Pad2): track 17.6 -> 18.8 mm
- net Net-(Rbin_U11-Pad1): track 12.8 -> 11.7 mm
- net Net-(Rbin_U9-Pad1): track 12.7 -> 11.7 mm
- net Net-(Rbin_U12-Pad1): track 21.1 -> 22.2 mm
- net Net-(Rbin_U10-Pad1): track 21.5 -> 22.3 mm
- net Net-(JPout_U3a1-Pad2): track 7.03 -> 6.46 mm
- net Net-(JPout_U4a1-Pad2): track 6.85 -> 6.28 mm
- net Net-(JPout_U2a1-Pad2): track 6.99 -> 6.42 mm

Commit message: board manufacturing changes
Connections:
- J_LDAC_SYNC_SCL_SDA1 pad 2: Net-(Udac1-Pad2) -> +5V
- TP_U2b1 pad 1: Net-(TP_U2b1-Pad1) -> +2V5
- TP_U3b1 pad 1: Net-(TP_U3b1-Pad1) -> +5V
- TP_U4a1 pad 1: Net-(TP_U4a1-Pad1) -> +2V5
- U2 pad 5: Net-(TP_U2b1-Pad1) -> +2V5
- U3 pad 5: Net-(TP_U3b1-Pad1) -> +5V
- U4 pad 3: Net-(TP_U4a1-Pad1) -> +2V5
- Udac1 pad 10: Net-(TP_U2b1-Pad1) -> +2V5
- Udac1 pad 2: Net-(Udac1-Pad2) -> +5V
- Udac1 pad 4: Net-(TP_U3b1-Pad1) -> +5V
- Udac1 pad 7: Net-(TP_U4a1-Pad1) -> +2V5
Routing:
- net +5V: track 506.1 -> 627.7 mm
- net +2V5: track 176.8 -> 291.2 mm
- net Net-(TP_U3b1-Pad1): track 108.3 -> 0.00 mm
- net Net-(TP_U2b1-Pad1): track 64.6 -> 0.00 mm
- net Net-(TP_U4a1-Pad1): track 49.1 -> 0.00 mm
- net Net-(Udac1-Pad2): track 12.1 -> 0.00 mm
- net -5V: track 404.8 -> 405.9 mm
Other:
- board outline added: 102.1 x 148.4 mm
- board text added: "TEST PCB - EEG"

Commit message: test with 2 dacs
Connections:
- J_LDAC_SYNC_SCL_SDA1 pad 2: +5V -> Net-(J_LDAC_SYNC_SCL_SDA1-Pad2)
- TP_U2b1 pad 1: +2V5 -> Net-(TP_U2b1-Pad1)
- TP_U3b1 pad 1: +5V -> Net-(TP_U3b1-Pad1)
- TP_U4a1 pad 1: +2V5 -> Net-(TP_U4a1-Pad1)
- U2 pad 5: +2V5 -> Net-(TP_U2b1-Pad1)
- U3 pad 5: +5V -> Net-(TP_U3b1-Pad1)
- U4 pad 3: +2V5 -> Net-(TP_U4a1-Pad1)
- Udac1 pad 10: +2V5 -> Net-(TP_U2b1-Pad1)
- Udac1 pad 2: +5V -> Net-(J_LDAC_SYNC_SCL_SDA1-Pad2)
- Udac1 pad 4: +5V -> Net-(TP_U3b1-Pad1)
- Udac1 pad 7: +2V5 -> Net-(TP_U4a1-Pad1)
Routing:
- net +5V: track 627.7 -> 506.1 mm
- net +2V5: track 291.2 -> 176.2 mm
- net Net-(TP_U3b1-Pad1): track 0.00 -> 108.3 mm
- net Net-(TP_U2b1-Pad1): track 0.00 -> 64.6 mm
- net Net-(TP_U4a1-Pad1): track 0.00 -> 49.1 mm
- net Net-(J_LDAC_SYNC_SCL_SDA1-Pad2): track 0.00 -> 12.1 mm
