File: KiCad/TestPCB/TestPCB.kicad_sch (KiCad schematic)
At the start: 91 parts, among them U1 MC33078, U10a1 OP07, U10b1 OP07, U11a1 OP07, U11b1 OP07, U12a1 OP07, U12b1 OP07, U2 MC33078, U3 MC33078, U4 MC33078, U5 OP07, U6 OP07, U7 OP07, U8 OP07, U9 TL431D, U9a1 OP07, U9b1 OP07

Commit message: First PCB run done
Connections:
- net at TP_U3a1.1, U3.3 (+): now also Udac1.5 (VOUTC); no longer Udac1.4 (VOUTA)
- net at TP_U3b1.1, U3.5 (+): now also Udac1.4 (VOUTA); no longer Udac1.5 (VOUTC)
- net at TP_U4a1.1, U4.3 (+): now also Udac1.7 (VOUTG); no longer Udac1.6 (VOUTE)
- net at TP_U4b1.1, U4.5 (+): now also Udac1.6 (VOUTE); no longer Udac1.7 (VOUTG)
Other:
- moved on the sheet: TP_U3a1, TP_U3b1, TP_U4a1, TP_U4b1
Changed lines of the file:
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@@
   (junction (at 161.925 70.485) (diameter 0) (color 0 0 0 0)
   )
-  (junction (at 95.25 184.785) (diameter 0) (color 0 0 0 0)
-  )
   (junction (at 185.42 195.58) (diameter 0) (color 0 0 0 0)
   )
@@
   (junction (at 117.475 33.02) (diameter 0) (color 0 0 0 0)
   )
-  (junction (at 93.98 146.05) (diameter 0) (color 0 0 0 0)
-  )
   (junction (at 100.965 102.235) (diameter 0) (color 0 0 0 0)
   )
@@
   (junction (at 162.56 220.98) (diameter 0) (color 0 0 0 0)
   )
-  (junction (at 92.71 107.315) (diameter 0) (color 0 0 0 0)
-  )
   (junction (at 182.245 20.955) (diameter 0) (color 0 0 0 0)
   )
-  (junction (at 96.52 223.52) (diameter 0) (color 0 0 0 0)
-  )
   (junction (at 117.475 218.44) (diameter 0) (color 0 0 0 0)
   )
   (junction (at 117.475 102.235) (diameter 0) (color 0 0 0 0)
   )
+  (junction (at 93.98 107.315) (diameter 0) (color 0 0 0 0)
+  )
   (junction (at 100.965 82.55) (diameter 0) (color 0 0 0 0)
   )
@@
   (junction (at 94.615 73.025) (diameter 0) (color 0 0 0 0)
   )
+  (junction (at 95.25 223.52) (diameter 0) (color 0 0 0 0)
+  )
   (junction (at 161.925 35.56) (diameter 0) (color 0 0 0 0)
   )
@@
   (junction (at 137.16 50.165) (diameter 0) (color 0 0 0 0)
   )
+  (junction (at 92.71 146.05) (diameter 0) (color 0 0 0 0)
+  )
   (junction (at 95.885 87.63) (diameter 0) (color 0 0 0 0)
   )
   (junction (at 177.165 94.615) (diameter 0) (color 0 0 0 0)
   )
+  (junction (at 96.52 184.785) (diameter 0) (color 0 0 0 0)
+  )
   (junction (at 71.12 104.775) (diameter 0) (color 0 0 0 0)
   )
@@
     (stroke (width 0) (type default) (color 0 0 0 0))
   )
+  (wire (pts (xy 95.25 94.615) (xy 95.25 223.52))
+    (stroke (width 0) (type default) (color 0 0 0 0))
+  )
   (wire (pts (xy 122.555 61.595) (xy 117.475 61.595))
     (stroke (width 0) (type default) (color 0 0 0 0))
@@
     (stroke (width 0) (type default) (color 0 0 0 0))
   )
-  (wire (pts (xy 92.71 84.455) (xy 92.71 107.315))
-    (stroke (width 0) (type default) (color 0 0 0 0))
-  )
   (wire (pts (xy 92.075 38.1) (xy 92.075 86.995))
     (stroke (width 0) (type default) (color 0 0 0 0))
   )
-  (wire (pts (xy 92.71 107.315) (xy 120.015 107.315))
-    (stroke (width 0) (type default) (color 0 0 0 0))
-  )
   (wire (pts (xy 149.225 104.775) (xy 153.035 104.775))
     (stroke (width 0) (type default) (color 0 0 0 0))
@@
     (stroke (width 0) (type default) (color 0 0 0 0))
   )
+  (wire (pts (xy 93.98 89.535) (xy 93.98 107.315))
+    (stroke (width 0) (type default) (color 0 0 0 0))
+  )
   (wire (pts (xy 92.075 38.1) (xy 120.015 38.1))
     (stroke (width 0) (type default) (color 0 0 0 0))
@@
     (stroke (width 0) (type default) (color 0 0 0 0))
   )
+  (wire (pts (xy 92.71 84.455) (xy 92.71 146.05))
+    (stroke (width 0) (type default) (color 0 0 0 0))
+  )
   (wire (pts (xy 187.325 28.575) (xy 189.865 28.575))
     (stroke (width 0) (type default) (color 0 0 0 0))
@@
     (stroke (width 0) (type default) (color 0 0 0 0))
   )
-  (wire (pts (xy 95.25 94.615) (xy 95.25 184.785))
-    (stroke (width 0) (type default) (color 0 0 0 0))
-  )
   (wire (pts (xy 184.15 40.64) (xy 184.15 33.02))
     (stroke (width 0) (type default) (color 0 0 0 0))
@@
     (stroke (width 0) (type default) (color 0 0 0 0))
   )
+  (wire (pts (xy 96.52 99.695) (xy 96.52 184.785))
+    (stroke (width 0) (type default) (color 0 0 0 0))
+  )
   (wire (pts (xy 114.3 102.235) (xy 117.475 102.235))
     (stroke (width 0) (type default) (color 0 0 0 0))
@@
     (stroke (width 0) (type default) (color 0 0 0 0))
   )
-  (wire (pts (xy 93.98 146.05) (xy 120.015 146.05))
+  (wire (pts (xy 92.71 146.05) (xy 120.015 146.05))
     (stroke (width 0) (type default) (color 0 0 0 0))
   )
-  (wire (pts (xy 120.015 223.52) (xy 96.52 223.52))
+  (wire (pts (xy 95.25 223.52) (xy 120.015 223.52))
     (stroke (width 0) (type default) (color 0 0 0 0))
   )
@@
     (stroke (width 0) (type default) (color 0 0 0 0))
   )
-  (wire (pts (xy 96.52 99.695) (xy 96.52 223.52))
-    (stroke (width 0) (type default) (color 0 0 0 0))
-  )
   (wire (pts (xy 117.475 61.595) (xy 117.475 67.945))
     (stroke (width 0) (type default) (color 0 0 0 0))
@@
     (stroke (width 0) (type default) (color 0 0 0 0))
   )
+  (wire (pts (xy 93.98 107.315) (xy 120.015 107.315))
+    (stroke (width 0) (type default) (color 0 0 0 0))
+  )
   (wire (pts (xy 161.925 104.775) (xy 167.005 104.775))
     (stroke (width 0) (type default) (color 0 0 0 0))
@@
     (stroke (width 0) (type default) (color 0 0 0 0))
   )
-  (wire (pts (xy 95.25 184.785) (xy 120.015 184.785))
+  (wire (pts (xy 96.52 184.785) (xy 120.015 184.785))
     (stroke (width 0) (type default) (color 0 0 0 0))
   )
@@
     (stroke (width 0) (type default) (color 0 0 0 0))
   )
-  (wire (pts (xy 93.98 89.535) (xy 93.98 146.05))
-    (stroke (width 0) (type default) (color 0 0 0 0))
-  )
   (wire (pts (xy 149.225 70.485) (xy 153.035 70.485))
     (stroke (width 0) (type default) (color 0 0 0 0))
@@
     (pin "1")
   )
-  (symbol (lib_id "Connector:TestPoint") (at 92.71 107.315 180) (unit 1)
+  (symbol (lib_id "Connector:TestPoint") (at 93.98 107.315 180) (unit 1)
     (in_bom yes) (on_board yes)
-    (property "Reference" "TP_U3a1" (id 0) (at 101.6 110.49 0)
+    (property "Reference" "TP_U3a1" (id 0) (at 102.87 110.49 0)
       (effects (font (size 1.27 1.27)) (justify left))
     )
-    (property "Value" "TestPoint" (id 1) (at 102.235 108.585 0)
+    (property "Value" "TestPoint" (id 1) (at 103.505 108.585 0)
       (effects (font (size 1.27 1.27)) (justify left))
     )
-    (property "Footprint" "TestPoint:TestPoint_Pad_4.0x4.0mm" (id 2) (at 87.63 107.315 0)
+    (property "Footprint" "TestPoint:TestPoint_Pad_4.0x4.0mm" (id 2) (at 88.9 107.315 0)
       (effects (font (size 1.27 1.27)) hide)
     )
-    (property "Datasheet" "~" (id 3) (at 87.63 107.315 0)
+    (property "Datasheet" "~" (id 3) (at 88.9 107.315 0)
       (effects (font (size 1.27 1.27)) hide)
     )
@@
     (pin "1")
   )
-  (symbol (lib_id "Connector:TestPoint") (at 93.98 146.05 180) (unit 1)
+  (symbol (lib_id "Connector:TestPoint") (at 92.71 146.05 180) (unit 1)
     (in_bom yes) (on_board yes)
-    (property "Reference" "TP_U3b1" (id 0) (at 102.87 149.225 0)
+    (property "Reference" "TP_U3b1" (id 0) (at 101.6 149.225 0)
       (effects (font (size 1.27 1.27)) (justify left))
     )
-    (property "Value" "TestPoint" (id 1) (at 103.505 147.32 0)
+    (property "Value" "TestPoint" (id 1) (at 102.235 147.32 0)
       (effects (font (size 1.27 1.27)) (justify left))
     )
-    (property "Footprint" "TestPoint:TestPoint_Pad_4.0x4.0mm" (id 2) (at 88.9 146.05 0)
+    (property "Footprint" "TestPoint:TestPoint_Pad_4.0x4.0mm" (id 2) (at 87.63 146.05 0)
       (effects (font (size 1.27 1.27)) hide)
     )
-    (property "Datasheet" "~" (id 3) (at 88.9 146.05 0)
+    (property "Datasheet" "~" (id 3) (at 87.63 146.05 0)
       (effects (font (size 1.27 1.27)) hide)
     )
@@
   (symbol (lib_id "power:+2V5") (at 52.07 33.02 0) (unit 1)
     (in_bom yes) (on_board yes) (fields_autoplaced)
-    (property "Reference" "#PWR?" (id 0) (at 52.07 36.83 0)
+    (property "Reference" "#PWR0155" (id 0) (at 52.07 36.83 0)
       (effects (font (size 1.27 1.27)) hide)
     )
@@
     (pin "1")
   )
-  (symbol (lib_id "Connector:TestPoint") (at 96.52 223.52 180) (unit 1)
+  (symbol (lib_id "Connector:TestPoint") (at 95.25 223.52 180) (unit 1)
     (in_bom yes) (on_board yes)
-    (property "Reference" "TP_U4b1" (id 0) (at 105.41 226.695 0)
+    (property "Reference" "TP_U4b1" (id 0) (at 104.14 226.695 0)
       (effects (font (size 1.27 1.27)) (justify left))
     )
-    (property "Value" "TestPoint" (id 1) (at 106.045 224.79 0)
+    (property "Value" "TestPoint" (id 1) (at 104.775 224.79 0)
       (effects (font (size 1.27 1.27)) (justify left))
     )
-    (property "Footprint" "TestPoint:TestPoint_Pad_4.0x4.0mm" (id 2) (at 91.44 223.52 0)
+    (property "Footprint" "TestPoint:TestPoint_Pad_4.0x4.0mm" (id 2) (at 90.17 223.52 0)
       (effects (font (size 1.27 1.27)) hide)
     )
-    (property "Datasheet" "~" (id 3) (at 91.44 223.52 0)
+    (property "Datasheet" "~" (id 3) (at 90.17 223.52 0)
       (effects (font (size 1.27 1.27)) hide)
     )
     (pin "1")
   )
-  (symbol (lib_id "Connector:TestPoint") (at 95.25 184.785 180) (unit 1)
+  (symbol (lib_id "Connector:TestPoint") (at 96.52 184.785 180) (unit 1)
     (in_bom yes) (on_board yes)
-    (property "Reference" "TP_U4a1" (id 0) (at 104.14 187.96 0)
+    (property "Reference" "TP_U4a1" (id 0) (at 105.41 187.96 0)
       (effects (font (size 1.27 1.27)) (justify left))
     )
-    (property "Value" "TestPoint" (id 1) (at 104.775 186.055 0)
+    (property "Value" "TestPoint" (id 1) (at 106.045 186.055 0)
       (effects (font (size 1.27 1.27)) (justify left))
     )
-    (property "Footprint" "TestPoint:TestPoint_Pad_4.0x4.0mm" (id 2) (at 90.17 184.785 0)
+    (property "Footprint" "TestPoint:TestPoint_Pad_4.0x4.0mm" (id 2) (at 91.44 184.785 0)
       (effects (font (size 1.27 1.27)) hide)
     )
-    (property "Datasheet" "~" (id 3) (at 90.17 184.785 0)
+    (property "Datasheet" "~" (id 3) (at 91.44 184.785 0)
       (effects (font (size 1.27 1.27)) hide)
     )
@@
     )
     (path "/5b1e363b-a2f1-47d0-afe9-9c06a609b4fb"
-      (reference "#PWR?") (unit 1) (value "+2V5") (footprint "")
+      (reference "#PWR0155") (unit 1) (value "+2V5") (footprint "")
     )
     (path "/3e3659d6-bafd-4943-b6ee-47a596b06d65"

Commit message: Added GND pins
Parts:
- added J1: (no value), symbol Connector:Conn_01x01_Male
- added J2: Conn_01x01_Male, symbol Connector:Conn_01x01_Male
Connections:
- net GND: now also J1.1 (Pin_1), J2.1 (Pin_1)
Changed lines of the file:
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@@
+    (pin "1")
+  )
+  (symbol (lib_id "Connector:Conn_01x01_Male") (at 73.66 49.53 0) (unit 1)
+    (in_bom yes) (on_board yes) (fields_autoplaced)
+    (property "Reference" "J2" (id 0) (at 74.295 43.815 0))
+    (property "Value" "Conn_01x01_Male" (id 1) (at 74.295 46.355 0))
+    (property "Footprint" "" (id 2) (at 73.66 49.53 0)
+      (effects (font (size 1.27 1.27)) hide)
+    )
+    (property "Datasheet" "~" (id 3) (at 73.66 49.53 0)
+      (effects (font (size 1.27 1.27)) hide)
+    )
     (pin "1")
   )
@@
     (pin "8")
   )
+  (symbol (lib_id "power:GND") (at 78.74 49.53 90) (unit 1)
+    (in_bom yes) (on_board yes) (fields_autoplaced)
+    (property "Reference" "#PWR0156" (id 0) (at 85.09 49.53 0)
+      (effects (font (size 1.27 1.27)) hide)
+    )
+    (property "Value" "GND" (id 1) (at 82.55 49.5299 90)
+      (effects (font (size 1.27 1.27)) (justify right))
+    )
+    (property "Footprint" "" (id 2) (at 78.74 49.53 0)
+      (effects (font (size 1.27 1.27)) hide)
+    )
+    (property "Datasheet" "" (id 3) (at 78.74 49.53 0)
+      (effects (font (size 1.27 1.27)) hide)
+    )
+    (pin "1")
+  )
   (symbol (lib_id "Connector:Conn_01x01_Male") (at 66.04 94.615 0) (unit 1)
     (in_bom yes) (on_board yes)
@@
     (pin "1")
   )
+  (symbol (lib_id "Connector:Conn_01x01_Male") (at 73.66 42.545 0) (unit 1)
+    (in_bom yes) (on_board yes) (fields_autoplaced)
+    (property "Reference" "J1" (id 0) (at 74.295 36.83 0))
+    (property "Value" "" (id 1) (at 74.295 39.37 0))
+    (property "Footprint" "" (id 2) (at 73.66 42.545 0)
+      (effects (font (size 1.27 1.27)) hide)
+    )
+    (property "Datasheet" "~" (id 3) (at 73.66 42.545 0)
+      (effects (font (size 1.27 1.27)) hide)
+    )
+    (pin "1")
+  )
   (symbol (lib_id "power:GND") (at 177.8 210.82 90) (mirror x) (unit 1)
     (in_bom yes) (on_board yes)
@@
     )
     (property "Datasheet" "" (id 3) (at 189.23 70.485 0)
+      (effects (font (size 1.27 1.27)) hide)
+    )
+    (pin "1")
+  )
+  (symbol (lib_id "power:GND") (at 78.74 42.545 90) (unit 1)
+    (in_bom yes) (on_board yes) (fields_autoplaced)
+    (property "Reference" "#PWR0157" (id 0) (at 85.09 42.545 0)
+      (effects (font (size 1.27 1.27)) hide)
+    )
+    (property "Value" "" (id 1) (at 82.55 42.5449 90)
+      (effects (font (size 1.27 1.27)) (justify right))
+    )
+    (property "Footprint" "" (id 2) (at 78.74 42.545 0)
+      (effects (font (size 1.27 1.27)) hide)
+    )
+    (property "Datasheet" "" (id 3) (at 78.74 42.545 0)
       (effects (font (size 1.27 1.27)) hide)
     )
@@
       (reference "#PWR0155") (unit 1) (value "+2V5") (footprint "")
     )
+    (path "/b9b57abf-7575-43d6-98ff-e2169e982f42"
+      (reference "#PWR0156") (unit 1) (value "GND") (footprint "")
+    )
+    (path "/ee910b77-e52f-4436-9f70-6a1a13124779"
+      (reference "#PWR0157") (unit 1) (value "GND") (footprint "")
+    )
     (path "/3e3659d6-bafd-4943-b6ee-47a596b06d65"
       (reference "Cref1") (unit 1) (value "100n") (footprint "Capacitor_THT:C_Disc_D5.0mm_W2.5mm_P5.00mm")
     )
+    (path "/e195398e-6848-402c-a5bd-e9ecc0f84f2b"
+      (reference "J1") (unit 1) (value "Conn_01x01_Male") (footprint "Connector_PinHeader_2.54mm:PinHeader_1x01_P2.54mm_Vertical")
+    )
+    (path "/2b48b6c3-f49a-4209-b24c-c98f096cd478"
+      (reference "J2") (unit 1) (value "Conn_01x01_Male") (footprint "Connector_PinHeader_2.54mm:PinHeader_1x01_P2.54mm_Vertical")
+    )
     (path "/f12ba46b-fd77-4f8a-8f8a-202b95bfd7d4"

Commit message: finished desing
Parts:
- removed J_LDAC1, J_SCL1, J_SDA1, J_SYNC1: Conn_01x01_Male, Connector_PinHeader_2.54mm:PinHeader_1x01_P2.54mm_Vertical, symbol Connector:Conn_01x01_Male
- added J_LDAC_SYNC_SCL_SDA1: (no value), symbol Connector:Conn_01x04_Male
- added TPRef2, TPRef3: Conn_01x01_Male, Connector_PinHeader_2.54mm:PinHeader_1x01_P2.54mm_Vertical, symbol Connector:Conn_01x01_Male
- Cref1: footprint Capacitor_THT:C_Disc_D5.0mm_W2.5mm_P5.00mm -> (none)
- J1: value (none) -> Conn_01x01_Male
- JPout_U1a1, JPout_U1b1, JPout_U2a1, JPout_U2b1, JPout_U3a1, JPout_U3b1, JPout_U4a1, JPout_U4b1: footprint Connector_PinHeader_2.54mm:PinHeader_1x02_P2.54mm_Vertical -> (none)
- Jout10a1, Jout10b1, Jout11a1, Jout11b1, Jout12a1, Jout12b1, Jout5, Jout6, Jout7, Jout8, Jout9a1, Jout9b1: footprint Connector_PinHeader_2.54mm:PinHeader_1x01_P2.54mm_Vertical -> (none)
- Rain_U10, Rain_U11, Rain_U12, Rain_U5, Rain_U6, Rain_U7, Rain_U8, Rain_U9, Rbin_U10, Rbin_U11, Rbin_U12, Rbin_U5, Rbin_U6, Rbin_U7, Rbin_U8, Rbin_U9, Rcin_U10, Rcin_U11, Rcin_U12, Rcin_U9: footprint Resistor_SMD:R_2010_5025Metric_Pad1.40x2.65mm_HandSolder -> (none)
- TPRef1: value (none) -> Conn_01x01_Male; footprint (none) -> Connector_PinHeader_2.54mm:PinHeader_1x01_P2.54mm_Vertical
- U10a1, U10b1, U11a1, U11b1, U12a1, U12b1, U5, U6, U7, U8, U9a1, U9b1: footprint (none) -> Package_DIP:DIP-8_W7.62mm_Socket_LongPads
Connections:
- net +5V: now also TPRef2.1 (Pin_1)
- net -5V: now also TPRef3.1 (Pin_1)
- net at Udac1.1 (~{LDAC}): now also J_LDAC_SYNC_SCL_SDA1.1 (Pin_1)
- net at R_SDA1.2, Udac1.15 (SDA): now also J_LDAC_SYNC_SCL_SDA1.4 (Pin_4)
- net at R_SCL1.2, Udac1.16 (SCL): now also J_LDAC_SYNC_SCL_SDA1.3 (Pin_3)
- net at Udac1.2 (ADDR0): now also J_LDAC_SYNC_SCL_SDA1.2 (Pin_2)

Commit message: Fixing PCB design
Parts:
- added JPin_U13b1, JPin_U1a1, JPin_U1b1, JPin_U2a1, JPin_U2b1, JPin_U3a1, JPin_U4a1, JPin_U4b1: Jumper_2_Bridged, Connector_PinHeader_2.54mm:PinHeader_1x02_P2.54mm_Vertical, symbol Jumper:Jumper_2_Bridged
- Cref1: footprint (none) -> Capacitor_THT:C_Disc_D5.0mm_W2.5mm_P2.50mm
- J_LDAC_SYNC_SCL_SDA1: value (none) -> Conn_01x04_Male
- Rain_U10, Rain_U11, Rain_U12, Rain_U5, Rain_U6, Rain_U7, Rain_U8, Rain_U9, Rbin_U10, Rbin_U11, Rbin_U12, Rbin_U5, Rbin_U6, Rbin_U7, Rbin_U8, Rbin_U9, Rcin_U10, Rcin_U11, Rcin_U12, Rcin_U9: footprint (none) -> Resistor_SMD:R_1206_3216Metric_Pad1.30x1.75mm_HandSolder
Connections:
- net at TP_U1a1.1, Udac1.13 (VOUTB): now also JPin_U1a1.1 (A); no longer U1.3 (+)
- net at TP_U1b1.1, Udac1.12 (VOUTD): now also JPin_U1b1.1 (A); no longer U1.5 (+)
- net at TP_U2b1.1, Udac1.10 (VOUTH): now also JPin_U2b1.1 (A); no longer U2.5 (+)
- net at TP_U2a1.1, Udac1.11 (VOUTF): now also JPin_U2a1.1 (A); no longer U2.3 (+)
- net at TP_U3b1.1, Udac1.4 (VOUTA): now also JPin_U13b1.1 (A); no longer U3.5 (+)
- net at TP_U3a1.1, Udac1.5 (VOUTC): now also JPin_U3a1.1 (A); no longer U3.3 (+)
- net at TP_U4b1.1, Udac1.6 (VOUTE): now also JPin_U4b1.1 (A); no longer U4.5 (+)
- net at TP_U4a1.1, Udac1.7 (VOUTG): now also JPin_U4a1.1 (A); no longer U4.3 (+)
- new net: JPin_U1a1.2 (B), U1.3 (+)
- new net: JPin_U1b1.2 (B), U1.5 (+)
- new net: JPin_U4b1.2 (B), U4.5 (+)
- new net: JPin_U2b1.2 (B), U2.5 (+)
- new net: JPin_U3a1.2 (B), U3.3 (+)
- new net: JPin_U4a1.2 (B), U4.3 (+)
- new net: JPin_U13b1.2 (B), U3.5 (+)
- new net: JPin_U2a1.2 (B), U2.3 (+)
Other:
- moved on the sheet: JPout_U1a1, JPout_U1b1, JPout_U2a1, JPout_U2b1, JPout_U3a1, JPout_U3b1, JPout_U4a1, JPout_U4b1, Jout10a1, Jout10b1, Jout11a1, Jout11b1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
