File: KiCad/TheBoard_2/TheBoard_2.kicad_pcb (KiCad board)
At the start: 2 copper layers, 150 x 100 mm, 48 parts, among them J1 Conn_01x03_Female, J2 Conn_01x03_Female, J3 Conn_01x16_Female, J4 Conn_01x36_Male, J5 Conn_01x16_Female, J6 Conn_01x02_Male, J7 USB_B_Micro, Q1 FS8205A, U1 MAX680CSA+T, U10 MCP6074-E/SL, U11 MCP6074-E/SL, U12 MCP6074-E/SL, U13 MCP6074-E/SL, U2 LM337_TO220, U3 MT3608, U4 TP4056, U5 DW01, U6 MCP6074-E/SL, U7 MCP6074-E/SL, U8 MCP6074-E/SL, U9 MCP6074-E/SL

Commit message: progress
Parts:
- removed C10: C, Capacitor_SMD:C_0603_1608Metric_Pad1.08x0.95mm_HandSolder
- removed C6, C7: C, Capacitor_SMD:C_1206_3216Metric
- removed C8, C9: C, Capacitor_SMD:C_0402_1005Metric_Pad0.74x0.62mm_HandSolder
- removed D1: D, Diode_SMD:D_SMA
- removed D2, D3: LED, LED_SMD:LED_0402_1005Metric_Pad0.77x0.64mm_HandSolder
- removed J7: USB_B_Micro, Connector_USB:USB_Micro-B_Molex_47346-0001
- removed L1: L, Inductor_SMD:L_10.4x10.4_H4.8
- removed Q1: FS8205A, Package_SO:TSSOP-8_4.4x3mm_P0.65mm
- removed RV2: R_Potentiometer, Potentiometer_THT:Potentiometer_Bourns_3296P_Horizontal
- added R10: R, Resistor_SMD:R_0805_2012Metric, F.Cu at (111.2, -64.0)
- added R100: R, Resistor_SMD:R_0805_2012Metric, F.Cu at (236.5, -36.0)
- added R101: R, Resistor_SMD:R_0805_2012Metric, F.Cu at (236.6, -40.6)
- added R102: R, Resistor_SMD:R_0805_2012Metric, F.Cu at (236.7, -45.4)
- added R103: R, Resistor_SMD:R_0805_2012Metric, F.Cu at (236.4, -55.0)
- added R104: R, Resistor_SMD:R_0805_2012Metric, F.Cu at (236.2, -59.9)
- added R105: R, Resistor_SMD:R_0805_2012Metric, F.Cu at (236.6, -64.7)
- added R106: R, Resistor_SMD:R_0805_2012Metric, F.Cu at (236.4, -69.4)
- added R107: R, Resistor_SMD:R_0805_2012Metric, F.Cu at (236.3, -73.3)
- added R108: R, Resistor_SMD:R_0805_2012Metric, F.Cu at (236.1, -78.3)
- added R109: R, Resistor_SMD:R_0805_2012Metric, F.Cu at (236.1, -82.3)
- added R11: R, Resistor_SMD:R_0805_2012Metric, F.Cu at (111.0, -58.1)
- added R110: R, Resistor_SMD:R_0805_2012Metric, F.Cu at (236.0, -86.2)
- added R111: R, Resistor_SMD:R_0805_2012Metric, F.Cu at (235.9, -90.4)
- added R112: R, Resistor_SMD:R_0805_2012Metric, F.Cu at (236.1, -94.7)
- added R113: R, Resistor_SMD:R_0805_2012Metric, F.Cu at (236.6, -50.5)
- added R114: R, Resistor_SMD:R_0805_2012Metric, F.Cu at (233.8, -26.9)
- added R115: R, Resistor_SMD:R_0805_2012Metric, F.Cu at (233.8, -31.8)
- added R116: R, Resistor_SMD:R_0805_2012Metric, F.Cu at (233.6, -36.8)
- added R117: R, Resistor_SMD:R_0805_2012Metric, F.Cu at (233.7, -41.4)
- added R118: R, Resistor_SMD:R_0805_2012Metric, F.Cu at (233.7, -46.3)
- added R119: R, Resistor_SMD:R_0805_2012Metric, F.Cu at (233.5, -56.0)
- added R12: R, Resistor_SMD:R_0805_2012Metric, F.Cu at (111.7, -51.2)
- added R120: R, Resistor_SMD:R_0805_2012Metric, F.Cu at (233.4, -60.9)
- added R121: R, Resistor_SMD:R_0805_2012Metric, F.Cu at (233.4, -65.6)
- added R122: R, Resistor_SMD:R_0805_2012Metric, F.Cu at (233.4, -70.2)
- added R123: R, Resistor_SMD:R_0805_2012Metric, F.Cu at (233.4, -74.2)
- added R124: R, Resistor_SMD:R_0805_2012Metric, F.Cu at (233.1, -79.2)
- added R125: R, Resistor_SMD:R_0805_2012Metric, F.Cu at (233.3, -82.9)
- added R126: R, Resistor_SMD:R_0805_2012Metric, F.Cu at (233.2, -87.0)
- added R127: R, Resistor_SMD:R_0805_2012Metric, F.Cu at (233.0, -91.2)
- added R128: R, Resistor_SMD:R_0805_2012Metric, F.Cu at (233.0, -95.5)
- added R129: R, Resistor_SMD:R_0805_2012Metric, F.Cu at (233.6, -51.4)
- added R13: R, Resistor_SMD:R_0805_2012Metric, F.Cu at (111.8, -46.1)
- added R14: R, Resistor_SMD:R_0805_2012Metric, F.Cu at (110.9, -38.8)
- added R15: R, Resistor_SMD:R_0805_2012Metric, F.Cu at (110.6, -31.3)
- added R16: R, Resistor_SMD:R_0805_2012Metric, F.Cu at (110.7, -25.1)
- added R17: R, Resistor_SMD:R_0805_2012Metric, F.Cu at (111.7, -87.5)
- added R18: R, Resistor_SMD:R_0805_2012Metric, F.Cu at (118.2, -110.8)
- added R19: R, Resistor_SMD:R_0805_2012Metric, F.Cu at (118.0, -105.5)
- added R20: R, Resistor_SMD:R_0805_2012Metric, F.Cu at (118.6, -99.2)
- added R21: R, Resistor_SMD:R_0805_2012Metric, F.Cu at (118.3, -94.0)
- added R22: R, Resistor_SMD:R_0805_2012Metric, F.Cu at (118.5, -88.1)
- added R23: R, Resistor_SMD:R_0805_2012Metric, F.Cu at (118.6, -82.4)
- added R24: R, Resistor_SMD:R_0805_2012Metric, F.Cu at (118.5, -77.2)
- added R25: R, Resistor_SMD:R_0805_2012Metric, F.Cu at (118.5, -71.4)
- added R26: R, Resistor_SMD:R_0805_2012Metric, F.Cu at (118.4, -64.0)
- added R27: R, Resistor_SMD:R_0805_2012Metric, F.Cu at (118.4, -58.6)
- added R28: R, Resistor_SMD:R_0805_2012Metric, F.Cu at (118.3, -51.8)
- added R29: R, Resistor_SMD:R_0805_2012Metric, F.Cu at (118.3, -45.9)
- added R30: R, Resistor_SMD:R_0805_2012Metric, F.Cu at (117.5, -39.0)
- added R31: R, Resistor_SMD:R_0805_2012Metric, F.Cu at (117.5, -31.7)
- added R32: R, Resistor_SMD:R_0805_2012Metric, F.Cu at (117.5, -25.9)
- added R33: R, Resistor_SMD:R_0805_2012Metric, F.Cu at (117.0, -18.6)
- added R34: R, Resistor_SMD:R_0805_2012Metric, F.Cu at (227.4, -26.9)
- added R35: R, Resistor_SMD:R_0805_2012Metric, F.Cu at (227.5, -31.7)
- added R36: R, Resistor_SMD:R_0805_2012Metric, F.Cu at (227.2, -36.4)
- added R37: R, Resistor_SMD:R_0805_2012Metric, F.Cu at (227.3, -41.1)
- added R38: R, Resistor_SMD:R_0805_2012Metric, F.Cu at (227.2, -46.1)
- added R39: R, Resistor_SMD:R_0805_2012Metric, F.Cu at (227.0, -51.5)
- added R40: R, Resistor_SMD:R_0805_2012Metric, F.Cu at (227.1, -55.9)
- added R41: R, Resistor_SMD:R_0805_2012Metric, F.Cu at (227.0, -60.6)
- added R42: R, Resistor_SMD:R_0805_2012Metric, F.Cu at (227.0, -65.5)
- added R43: R, Resistor_SMD:R_0805_2012Metric, F.Cu at (226.6, -70.1)
- added R44: R, Resistor_SMD:R_0805_2012Metric, F.Cu at (226.5, -74.3)
- added R45: R, Resistor_SMD:R_0805_2012Metric, F.Cu at (226.1, -79.3)
- added R46: R, Resistor_SMD:R_0805_2012Metric, F.Cu at (225.8, -82.8)
- added R47: R, Resistor_SMD:R_0805_2012Metric, F.Cu at (225.7, -86.9)
- added R48: R, Resistor_SMD:R_0805_2012Metric, F.Cu at (225.7, -90.9)
- added R49: R, Resistor_SMD:R_0805_2012Metric, F.Cu at (225.7, -95.3)
- added R50: R, Resistor_SMD:R_0805_2012Metric, F.Cu at (220.7, -45.9)
- added R51: R, Resistor_SMD:R_0805_2012Metric, F.Cu at (221.1, -27.0)
- added R52: R, Resistor_SMD:R_0805_2012Metric, F.Cu at (220.8, -31.5)
- added R53: R, Resistor_SMD:R_0805_2012Metric, F.Cu at (220.7, -36.4)
- added R54: R, Resistor_SMD:R_0805_2012Metric, F.Cu at (220.6, -41.0)
- added R55: R, Resistor_SMD:R_0805_2012Metric, F.Cu at (220.7, -51.4)
- added R56: R, Resistor_SMD:R_0805_2012Metric, F.Cu at (220.7, -56.3)
- added R57: R, Resistor_SMD:R_0805_2012Metric, F.Cu at (220.6, -60.6)
- added R58: R, Resistor_SMD:R_0805_2012Metric, F.Cu at (220.5, -65.4)
- added R59: R, Resistor_SMD:R_0805_2012Metric, F.Cu at (220.3, -70.1)
- added R60: R, Resistor_SMD:R_0805_2012Metric, F.Cu at (220.3, -74.6)
- added R61: R, Resistor_SMD:R_0805_2012Metric, F.Cu at (220.1, -79.4)
- added R62: R, Resistor_SMD:R_0805_2012Metric, F.Cu at (219.9, -82.6)
- added R63: R, Resistor_SMD:R_0805_2012Metric, F.Cu at (219.8, -86.8)
- added R64: R, Resistor_SMD:R_0805_2012Metric, F.Cu at (219.4, -91.0)
- added R65: R, Resistor_SMD:R_0805_2012Metric, F.Cu at (219.4, -95.2)
- added R66: R, Resistor_SMD:R_0805_2012Metric, F.Cu at (125.5, -82.7)
- added R67: R, Resistor_SMD:R_0805_2012Metric, F.Cu at (124.6, -110.9)
- added R68: R, Resistor_SMD:R_0805_2012Metric, F.Cu at (124.6, -105.5)
- added R69: R, Resistor_SMD:R_0805_2012Metric, F.Cu at (124.6, -99.3)
- added R70: R, Resistor_SMD:R_0805_2012Metric, F.Cu at (125.3, -93.9)
- added R71: R, Resistor_SMD:R_0805_2012Metric, F.Cu at (125.4, -88.5)
- added R72: R, Resistor_SMD:R_0805_2012Metric, F.Cu at (124.7, -77.4)
- added R73: R, Resistor_SMD:R_0805_2012Metric, F.Cu at (124.9, -71.4)
- added R74: R, Resistor_SMD:R_0805_2012Metric, F.Cu at (124.8, -64.2)
- added R75: R, Resistor_SMD:R_0805_2012Metric, F.Cu at (124.7, -58.2)
- added R76: R, Resistor_SMD:R_0805_2012Metric, F.Cu at (124.7, -51.8)
- added R77: R, Resistor_SMD:R_0805_2012Metric, F.Cu at (124.6, -46.1)
- added R78: R, Resistor_SMD:R_0805_2012Metric, F.Cu at (124.4, -38.7)
- added R79: R, Resistor_SMD:R_0805_2012Metric, F.Cu at (124.0, -31.9)
- added R8: R, Resistor_SMD:R_0805_2012Metric, F.Cu at (111.9, -77.0)
- added R80: R, Resistor_SMD:R_0805_2012Metric, F.Cu at (123.7, -26.1)
- added R81: R, Resistor_SMD:R_0805_2012Metric, F.Cu at (123.8, -18.6)
- added R82: R, Resistor_SMD:R_0805_2012Metric, F.Cu at (128.3, -81.8)
- added R83: R, Resistor_SMD:R_0805_2012Metric, F.Cu at (127.7, -110.0)
- added R84: R, Resistor_SMD:R_0805_2012Metric, F.Cu at (127.6, -104.7)
- added R85: R, Resistor_SMD:R_0805_2012Metric, F.Cu at (127.5, -98.5)
- added R86: R, Resistor_SMD:R_0805_2012Metric, F.Cu at (128.2, -93.2)
- added R87: R, Resistor_SMD:R_0805_2012Metric, F.Cu at (128.4, -87.7)
- added R88: R, Resistor_SMD:R_0805_2012Metric, F.Cu at (127.6, -76.6)
- added R89: R, Resistor_SMD:R_0805_2012Metric, F.Cu at (127.8, -70.6)
- added R9: R, Resistor_SMD:R_0805_2012Metric, F.Cu at (111.4, -71.2)
- added R90: R, Resistor_SMD:R_0805_2012Metric, F.Cu at (127.8, -63.4)
- added R91: R, Resistor_SMD:R_0805_2012Metric, F.Cu at (127.9, -57.3)
- added R92: R, Resistor_SMD:R_0805_2012Metric, F.Cu at (127.8, -50.9)
- added R93: R, Resistor_SMD:R_0805_2012Metric, F.Cu at (127.6, -45.3)
- added R94: R, Resistor_SMD:R_0805_2012Metric, F.Cu at (127.3, -37.8)
- added R95: R, Resistor_SMD:R_0805_2012Metric, F.Cu at (127.1, -31.1)
- added R96: R, Resistor_SMD:R_0805_2012Metric, F.Cu at (126.9, -25.4)
- added R97: R, Resistor_SMD:R_0805_2012Metric, F.Cu at (126.8, -17.8)
- added R98: R, Resistor_SMD:R_0805_2012Metric, F.Cu at (236.8, -26.1)
- added R99: R, Resistor_SMD:R_0805_2012Metric, F.Cu at (236.7, -30.9)
- added U14: LM2902, Package_SO:SOIC-14_3.9x8.7mm_P1.27mm, F.Cu at (100.6, 78.7)
- added U19: LM2902, Package_SO:SOIC-14_3.9x8.7mm_P1.27mm, F.Cu at (209.5, 112.8)
- added U20: LM2902, Package_SO:SOIC-14_3.9x8.7mm_P1.27mm, F.Cu at (209.5, 101.4)
- added U21: LM2902, Package_SO:SOIC-14_3.9x8.7mm_P1.27mm, F.Cu at (209.4, 90.8)
- added U22: LM2902, Package_SO:SOIC-14_3.9x8.7mm_P1.27mm, F.Cu at (209.3, 80.0)
- R1, R4, R5, R6, R7: footprint Resistor_SMD:R_0402_1005Metric_Pad0.72x0.64mm_HandSolder -> Resistor_SMD:R_0805_2012Metric
- U3: value MT3608 -> LM2902; footprint Package_TO_SOT_SMD:SOT-23-6 -> Package_SO:SOIC-14_3.9x8.7mm_P1.27mm
- U4: value TP4056 -> LM2902; footprint Package_SO:SOIC-8-1EP_3.9x4.9mm_P1.27mm_EP2.29x3mm -> Package_SO:SOIC-14_3.9x8.7mm_P1.27mm
- U5: value DW01 -> LM2902; footprint Package_TO_SOT_SMD:SOT-23-6_Handsoldering -> Package_SO:SOIC-14_3.9x8.7mm_P1.27mm
- moved R3 184.5 mm to (111.9, -110.5), turned to 0 degrees
- moved R5 168.4 mm to (111.8, -99.0), turned to 0 degrees
- moved R4 164.4 mm to (111.4, -105.3), turned to 0 degrees
- moved R6 161.4 mm to (111.7, -93.7), turned to 0 degrees
- moved R7 139.7 mm to (111.9, -82.0), turned to 0 degrees
- moved U3 83.9 mm to (100.7, 116.4)
- moved R1 79.4 mm to (110.0, -18.9), turned to 0 degrees
- moved U6 78.5 mm to (192.5, 127.2)
- moved U9 59.2 mm to (164.0, 127.4)
- moved U1 56.9 mm to (144.4, 25.5)
- moved C1 56.9 mm to (149.2, 19.5)
- moved C2 56.9 mm to (138.5, 28.1)
- moved C3 56.9 mm to (138.5, 34.3)
- moved C4 56.9 mm to (154.2, 40.0)
- moved C5 56.9 mm to (163.0, 20.6)
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Connections:
- J3 pad 1: unconnected-(J3-Pad1) -> Net-(J3-Pad1)
- J3 pad 10: unconnected-(J3-Pad10) -> Net-(J3-Pad10)
- J3 pad 11: unconnected-(J3-Pad11) -> Net-(J3-Pad11)
- J3 pad 12: unconnected-(J3-Pad12) -> Net-(J3-Pad12)
- J3 pad 13: unconnected-(J3-Pad13) -> Net-(J3-Pad13)
- J3 pad 14: unconnected-(J3-Pad14) -> Net-(J3-Pad14)
- J3 pad 15: unconnected-(J3-Pad15) -> Net-(J3-Pad15)
- J3 pad 16: unconnected-(J3-Pad16) -> Net-(J3-Pad16)
- J3 pad 2: unconnected-(J3-Pad2) -> Net-(J3-Pad2)
- J3 pad 3: unconnected-(J3-Pad3) -> Net-(J3-Pad3)
- J3 pad 4: unconnected-(J3-Pad4) -> Net-(J3-Pad4)
- J3 pad 5: unconnected-(J3-Pad5) -> Net-(J3-Pad5)
- J3 pad 6: unconnected-(J3-Pad6) -> Net-(J3-Pad6)
- J3 pad 7: unconnected-(J3-Pad7) -> Net-(J3-Pad7)
- J3 pad 8: unconnected-(J3-Pad8) -> Net-(J3-Pad8)
- J3 pad 9: unconnected-(J3-Pad9) -> Net-(J3-Pad9)
- J4 pad 10: unconnected-(J4-Pad10) -> Net-(J4-Pad10)
- J4 pad 11: unconnected-(J4-Pad11) -> Net-(J4-Pad11)
- J4 pad 12: unconnected-(J4-Pad12) -> Net-(J4-Pad12)
- J4 pad 13: unconnected-(J4-Pad13) -> Net-(J4-Pad13)
- J4 pad 14: unconnected-(J4-Pad14) -> Net-(J4-Pad14)
- J4 pad 15: unconnected-(J4-Pad15) -> Net-(J4-Pad15)
- J4 pad 16: unconnected-(J4-Pad16) -> Net-(J4-Pad16)
- J4 pad 17: unconnected-(J4-Pad17) -> Net-(J4-Pad17)
- J4 pad 18: unconnected-(J4-Pad18) -> Net-(J4-Pad18)
- J4 pad 19: unconnected-(J4-Pad19) -> Net-(J4-Pad19)
- J4 pad 20: unconnected-(J4-Pad20) -> Net-(J4-Pad20)
- J4 pad 21: unconnected-(J4-Pad21) -> Net-(J4-Pad21)
- J4 pad 22: unconnected-(J4-Pad22) -> Net-(J4-Pad22)
- J4 pad 23: unconnected-(J4-Pad23) -> Net-(J4-Pad23)
- J4 pad 24: unconnected-(J4-Pad24) -> Net-(J4-Pad24)
- J4 pad 25: unconnected-(J4-Pad25) -> Net-(J4-Pad25)
- J4 pad 26: unconnected-(J4-Pad26) -> Net-(J4-Pad26)
- J4 pad 27: unconnected-(J4-Pad27) -> Net-(J4-Pad27)
- J4 pad 28: unconnected-(J4-Pad28) -> Net-(J4-Pad28)
- J4 pad 29: unconnected-(J4-Pad29) -> Net-(J4-Pad29)
- J4 pad 3: unconnected-(J4-Pad3) -> Net-(J4-Pad3)
- J4 pad 30: unconnected-(J4-Pad30) -> Net-(J4-Pad30)
- J4 pad 31: unconnected-(J4-Pad31) -> Net-(J4-Pad31)
- J4 pad 32: unconnected-(J4-Pad32) -> Net-(J4-Pad32)
- J4 pad 33: unconnected-(J4-Pad33) -> Net-(J4-Pad33)
- J4 pad 34: unconnected-(J4-Pad34) -> Net-(J4-Pad34)
- J4 pad 4: unconnected-(J4-Pad4) -> Net-(J4-Pad4)
- J4 pad 5: unconnected-(J4-Pad5) -> Net-(J4-Pad5)
- J4 pad 6: unconnected-(J4-Pad6) -> Net-(J4-Pad6)
- J4 pad 7: unconnected-(J4-Pad7) -> Net-(J4-Pad7)
- J4 pad 8: unconnected-(J4-Pad8) -> Net-(J4-Pad8)
- J4 pad 9: unconnected-(J4-Pad9) -> Net-(J4-Pad9)
- J5 pad 1: unconnected-(J5-Pad1) -> Net-(J5-Pad1)
- J5 pad 10: unconnected-(J5-Pad10) -> Net-(J5-Pad10)
- J5 pad 11: unconnected-(J5-Pad11) -> Net-(J5-Pad11)
- J5 pad 12: unconnected-(J5-Pad12) -> Net-(J5-Pad12)
- J5 pad 13: unconnected-(J5-Pad13) -> Net-(J5-Pad13)
- J5 pad 14: unconnected-(J5-Pad14) -> Net-(J5-Pad14)
- J5 pad 15: unconnected-(J5-Pad15) -> Net-(J5-Pad15)
- J5 pad 16: unconnected-(J5-Pad16) -> Net-(J5-Pad16)
- J5 pad 2: unconnected-(J5-Pad2) -> Net-(J5-Pad2)
- J5 pad 3: unconnected-(J5-Pad3) -> Net-(J5-Pad3)
- J5 pad 4: unconnected-(J5-Pad4) -> Net-(J5-Pad4)
- J5 pad 5: unconnected-(J5-Pad5) -> Net-(J5-Pad5)
- J5 pad 6: unconnected-(J5-Pad6) -> Net-(J5-Pad6)
- J5 pad 7: unconnected-(J5-Pad7) -> Net-(J5-Pad7)
- J5 pad 8: unconnected-(J5-Pad8) -> Net-(J5-Pad8)
- J5 pad 9: unconnected-(J5-Pad9) -> Net-(J5-Pad9)
- R1 pad 1: Net-(D2-Pad1) -> +2V5
- R3 pad 1: Net-(R3-Pad1) -> +2V5
- R3 pad 2: GND -> Net-(R18-Pad1)
- R4 pad 1: Net-(D3-Pad1) -> +2V5
- R4 pad 2: Net-(R4-Pad2) -> Net-(R19-Pad1)
- R5 pad 1: Net-(R5-Pad1) -> +2V5
- R5 pad 2: GND -> Net-(R20-Pad1)
- R6 pad 1: Net-(R6-Pad1) -> +2V5
- R6 pad 2: GND -> Net-(R21-Pad1)
- R7 pad 1: Net-(C9-Pad1) -> +2V5
- R7 pad 2: OUT/B+ -> Net-(R23-Pad1)
- U10 pad 1: unconnected-(U10-Pad1) -> Net-(J4-Pad22)
- U10 pad 10: unconnected-(U10-Pad10) -> Net-(R115-Pad2)
- U10 pad 11: unconnected-(U10-Pad11) -> -5V
- U10 pad 12: unconnected-(U10-Pad12) -> Net-(R114-Pad2)
- U10 pad 13: unconnected-(U10-Pad13) -> Net-(J4-Pad19)
- U10 pad 14: unconnected-(U10-Pad14) -> Net-(J4-Pad19)
- U10 pad 2: unconnected-(U10-Pad2) -> Net-(J4-Pad22)
- U10 pad 3: unconnected-(U10-Pad3) -> Net-(R101-Pad2)
- U10 pad 4: unconnected-(U10-Pad4) -> +5V
- U10 pad 5: unconnected-(U10-Pad5) -> Net-(R100-Pad2)
- U10 pad 6: unconnected-(U10-Pad6) -> Net-(J4-Pad21)
- U10 pad 7: unconnected-(U10-Pad7) -> Net-(J4-Pad21)
- U10 pad 8: unconnected-(U10-Pad8) -> Net-(J4-Pad20)
- U10 pad 9: unconnected-(U10-Pad9) -> Net-(J4-Pad20)
- U11 pad 1: unconnected-(U11-Pad1) -> Net-(J4-Pad26)
- U11 pad 10: unconnected-(U11-Pad10) -> Net-(R113-Pad2)
- U11 pad 11: unconnected-(U11-Pad11) -> -5V
- U11 pad 12: unconnected-(U11-Pad12) -> Net-(R102-Pad2)
- U11 pad 13: unconnected-(U11-Pad13) -> Net-(J4-Pad23)
- U11 pad 14: unconnected-(U11-Pad14) -> Net-(J4-Pad23)
- U11 pad 2: unconnected-(U11-Pad2) -> Net-(J4-Pad26)
- U11 pad 3: unconnected-(U11-Pad3) -> Net-(R104-Pad2)
- U11 pad 4: unconnected-(U11-Pad4) -> +5V
- U11 pad 5: unconnected-(U11-Pad5) -> Net-(R103-Pad2)
- U11 pad 6: unconnected-(U11-Pad6) -> Net-(J4-Pad25)
- U11 pad 7: unconnected-(U11-Pad7) -> Net-(J4-Pad25)
- U11 pad 8: unconnected-(U11-Pad8) -> Net-(J4-Pad24)
- U11 pad 9: unconnected-(U11-Pad9) -> Net-(J4-Pad24)
- U12 pad 1: unconnected-(U12-Pad1) -> Net-(J4-Pad30)
- U12 pad 10: unconnected-(U12-Pad10) -> Net-(R106-Pad2)
- U12 pad 11: unconnected-(U12-Pad11) -> -5V
- U12 pad 12: unconnected-(U12-Pad12) -> Net-(R105-Pad2)
- U12 pad 13: unconnected-(U12-Pad13) -> Net-(J4-Pad27)
- U12 pad 14: unconnected-(U12-Pad14) -> Net-(J4-Pad27)
- U12 pad 2: unconnected-(U12-Pad2) -> Net-(J4-Pad30)
- U12 pad 3: unconnected-(U12-Pad3) -> Net-(R108-Pad2)
- U12 pad 4: unconnected-(U12-Pad4) -> +5V
- U12 pad 5: unconnected-(U12-Pad5) -> Net-(R107-Pad2)
- U12 pad 6: unconnected-(U12-Pad6) -> Net-(J4-Pad29)
- U12 pad 7: unconnected-(U12-Pad7) -> Net-(J4-Pad29)
- U12 pad 8: unconnected-(U12-Pad8) -> Net-(J4-Pad28)
- U12 pad 9: unconnected-(U12-Pad9) -> Net-(J4-Pad28)
- U13 pad 1: unconnected-(U13-Pad1) -> Net-(J4-Pad34)
- U13 pad 10: unconnected-(U13-Pad10) -> Net-(R110-Pad2)
- U13 pad 11: unconnected-(U13-Pad11) -> -5V
- U13 pad 12: unconnected-(U13-Pad12) -> Net-(R109-Pad2)
- U13 pad 13: unconnected-(U13-Pad13) -> Net-(J4-Pad31)
- U13 pad 14: unconnected-(U13-Pad14) -> Net-(J4-Pad31)
- U13 pad 2: unconnected-(U13-Pad2) -> Net-(J4-Pad34)
- U13 pad 3: unconnected-(U13-Pad3) -> Net-(R112-Pad2)
- U13 pad 4: unconnected-(U13-Pad4) -> +5V
- U13 pad 5: unconnected-(U13-Pad5) -> Net-(R111-Pad2)
- U13 pad 6: unconnected-(U13-Pad6) -> Net-(J4-Pad33)
- U13 pad 7: unconnected-(U13-Pad7) -> Net-(J4-Pad33)
- U13 pad 8: unconnected-(U13-Pad8) -> Net-(J4-Pad32)
- U13 pad 9: unconnected-(U13-Pad9) -> Net-(J4-Pad32)
- U3 pad 2: GND -> Net-(R18-Pad1)
- U3 pad 3: Net-(R3-Pad1) -> Net-(J5-Pad16)
- U3 pad 4: unconnected-(U3-Pad4) -> +5V
- U3 pad 5: Net-(C6-Pad1) -> Net-(J5-Pad15)
- U3 pad 6: unconnected-(U3-Pad6) -> Net-(R19-Pad1)
- U4 pad 1: GND -> Net-(R22-Pad2)
- U4 pad 2: Net-(R5-Pad1) -> Net-(R17-Pad2)
- U4 pad 3: GND -> Net-(J5-Pad12)
- U4 pad 4: Net-(C8-Pad1) -> +5V
- U4 pad 5: OUT/B+ -> Net-(J5-Pad11)
- U4 pad 6: Net-(R4-Pad2) -> Net-(R23-Pad1)
- U4 pad 7: Net-(R1-Pad2) -> Net-(R23-Pad2)
- U4 pad 8: Net-(C8-Pad1) -> Net-(R24-Pad2)
- U4 pad 9: unconnected-(U4-Pad9) -> Net-(R24-Pad1)
- U5 pad 2: Net-(R6-Pad1) -> Net-(R10-Pad2)
- U5 pad 3: Net-(Q1-Pad5) -> Net-(J5-Pad8)
- U5 pad 4: unconnected-(U5-Pad4) -> +5V
- U5 pad 5: Net-(C9-Pad1) -> Net-(J5-Pad7)
- U5 pad 6: B- -> Net-(R11-Pad2)
- U6 pad 1: unconnected-(U6-Pad1) -> Net-(J4-Pad6)
- U6 pad 10: unconnected-(U6-Pad10) -> Net-(R80-Pad2)
- U6 pad 11: unconnected-(U6-Pad11) -> -5V
- U6 pad 12: unconnected-(U6-Pad12) -> Net-(R81-Pad2)
- U6 pad 13: unconnected-(U6-Pad13) -> Net-(J4-Pad3)
- U6 pad 14: unconnected-(U6-Pad14) -> Net-(J4-Pad3)
- U6 pad 2: unconnected-(U6-Pad2) -> Net-(J4-Pad6)
- U6 pad 3: unconnected-(U6-Pad3) -> Net-(R78-Pad2)
- U6 pad 4: unconnected-(U6-Pad4) -> +5V
- U6 pad 5: unconnected-(U6-Pad5) -> Net-(R79-Pad2)
- U6 pad 6: unconnected-(U6-Pad6) -> Net-(J4-Pad5)
- U6 pad 7: unconnected-(U6-Pad7) -> Net-(J4-Pad5)
- U6 pad 8: unconnected-(U6-Pad8) -> Net-(J4-Pad4)
- U6 pad 9: unconnected-(U6-Pad9) -> Net-(J4-Pad4)
- U7 pad 1: unconnected-(U7-Pad1) -> Net-(J4-Pad10)
- U7 pad 10: unconnected-(U7-Pad10) -> Net-(R76-Pad2)
- U7 pad 11: unconnected-(U7-Pad11) -> -5V
- U7 pad 12: unconnected-(U7-Pad12) -> Net-(R77-Pad2)
- U7 pad 13: unconnected-(U7-Pad13) -> Net-(J4-Pad7)
- U7 pad 14: unconnected-(U7-Pad14) -> Net-(J4-Pad7)
- U7 pad 2: unconnected-(U7-Pad2) -> Net-(J4-Pad10)
- U7 pad 3: unconnected-(U7-Pad3) -> Net-(R74-Pad2)
- U7 pad 4: unconnected-(U7-Pad4) -> +5V
- U7 pad 5: unconnected-(U7-Pad5) -> Net-(R75-Pad2)
- U7 pad 6: unconnected-(U7-Pad6) -> Net-(J4-Pad9)
- U7 pad 7: unconnected-(U7-Pad7) -> Net-(J4-Pad9)
- U7 pad 8: unconnected-(U7-Pad8) -> Net-(J4-Pad8)
- U7 pad 9: unconnected-(U7-Pad9) -> Net-(J4-Pad8)
- U8 pad 1: unconnected-(U8-Pad1) -> Net-(J4-Pad14)
- U8 pad 10: unconnected-(U8-Pad10) -> Net-(R72-Pad2)
- U8 pad 12: unconnected-(U8-Pad12) -> Net-(R73-Pad2)
- U8 pad 13: unconnected-(U8-Pad13) -> Net-(J4-Pad11)
- U8 pad 14: unconnected-(U8-Pad14) -> Net-(J4-Pad11)
- U8 pad 2: unconnected-(U8-Pad2) -> Net-(J4-Pad14)
- U8 pad 3: unconnected-(U8-Pad3) -> Net-(R71-Pad2)
- U8 pad 4: unconnected-(U8-Pad4) -> +5V
- U8 pad 5: unconnected-(U8-Pad5) -> Net-(R66-Pad2)
- U8 pad 6: unconnected-(U8-Pad6) -> Net-(J4-Pad13)
- U8 pad 7: unconnected-(U8-Pad7) -> Net-(J4-Pad13)
- U8 pad 8: unconnected-(U8-Pad8) -> Net-(J4-Pad12)
- U8 pad 9: unconnected-(U8-Pad9) -> Net-(J4-Pad12)
- U9 pad 1: unconnected-(U9-Pad1) -> Net-(J4-Pad18)
- U9 pad 10: unconnected-(U9-Pad10) -> Net-(R69-Pad2)
- U9 pad 11: unconnected-(U9-Pad11) -> -5V
- U9 pad 12: unconnected-(U9-Pad12) -> Net-(R70-Pad2)
- U9 pad 13: unconnected-(U9-Pad13) -> Net-(J4-Pad15)
- U9 pad 14: unconnected-(U9-Pad14) -> Net-(J4-Pad15)
- U9 pad 2: unconnected-(U9-Pad2) -> Net-(J4-Pad18)
- U9 pad 3: unconnected-(U9-Pad3) -> Net-(R67-Pad2)
- U9 pad 4: unconnected-(U9-Pad4) -> +5V
- U9 pad 5: unconnected-(U9-Pad5) -> Net-(R68-Pad2)
- U9 pad 6: unconnected-(U9-Pad6) -> Net-(J4-Pad17)
- U9 pad 7: unconnected-(U9-Pad7) -> Net-(J4-Pad17)
- U9 pad 8: unconnected-(U9-Pad8) -> Net-(J4-Pad16)
- U9 pad 9: unconnected-(U9-Pad9) -> Net-(J4-Pad16)
Routing:
- net GND: track 41.3 -> 0.00 mm
- net Net-(C8-Pad1): track 29.5 -> 0.00 mm, vias 2 -> 0
- net Net-(C7-Pad1): track 17.3 -> 0.00 mm
- net Net-(R18-Pad2): track 16.0 -> 0.00 mm
- net Net-(R3-Pad1): track 15.8 -> 0.00 mm
- net B-: track 15.1 -> 0.00 mm
- net unconnected-(J7-Pad6): track 12.6 -> 0.00 mm
- net Net-(C6-Pad1): track 12.0 -> 0.00 mm
- net OUT/B+: track 10.7 -> 0.00 mm
- net Net-(Q1-Pad5): track 9.62 -> 0.00 mm, vias 2 -> 0
- net Net-(R6-Pad1): track 8.22 -> 0.00 mm, vias 2 -> 0
- net Net-(C9-Pad1): track 8.12 -> 0.00 mm
- net Net-(Q1-Pad1): track 5.74 -> 0.00 mm
- net Net-(R1-Pad2): track 3.23 -> 0.00 mm
- net Net-(R4-Pad2): track 3.14 -> 0.00 mm
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