File: KiCad/TheBoard_2/TheBoard_2.kicad_pcb (KiCad board)
At the start: 2 copper layers, 150 x 100 mm, 163 parts, among them J1 Conn_01x03_Female, J2 Conn_01x03_Female, J3 Conn_01x16_Female, J4 Conn_01x36_Male, J5 Conn_01x16_Female, J6 Conn_01x02_Male, U1 MAX680CSA+T, U10 MCP6074-E/SL, U11 MCP6074-E/SL, U12 MCP6074-E/SL, U13 MCP6074-E/SL, U14 LM2902, U19 LM2902, U2 LM337_TO220, U20 LM2902, U21 LM2902, U22 LM2902, U3 LM2902, U4 LM2902, U5 LM2902, U6 MCP6074-E/SL, U7 MCP6074-E/SL, U8 MCP6074-E/SL, U9 MCP6074-E/SL

Commit message: board2 progress
Parts:
- J4: footprint Connector_PinHeader_2.54mm:PinHeader_2x18_P2.54mm_Horizontal -> Connector_PinHeader_2.54mm:PinHeader_1x36_P2.54mm_Horizontal
- moved R83 232.6 mm to (107.0, 121.7), turned to 0 degrees
- moved R112 231.1 mm to (155.5, 121.9), turned to 0 degrees
- moved R67 230.1 mm to (108.0, 118.6), turned to -90 degrees
- moved R84 228.6 mm to (96.0, 121.8), turned to 0 degrees
- moved R128 227.6 mm to (156.3, 118.8), turned to -90 degrees
- moved R68 225.9 mm to (96.9, 118.7), turned to -90 degrees
- moved R111 224.5 mm to (162.8, 121.8), turned to 0 degrees
- moved R85 222.0 mm to (99.8, 121.7), turned to 0 degrees
- moved R127 221.3 mm to (163.6, 118.9), turned to -90 degrees
- moved R19 220.1 mm to (96.8, 113.6), turned to -90 degrees
- moved R69 219.5 mm to (100.6, 118.8), turned to -90 degrees
- moved R110 219.3 mm to (166.5, 121.8), turned to 0 degrees
- moved R3 218.7 mm to (94.1, 107.4)
- moved R4 218.7 mm to (94.1, 112.6)
- moved R18 218.3 mm to (96.8, 106.4), turned to 90 degrees
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Connections:
- R102 pad 2: Net-(R102-Pad2) -> Net-(U7-Pad5)
- R103 pad 2: Net-(R103-Pad2) -> Net-(U7-Pad12)
- R105 pad 2: Net-(R105-Pad2) -> Net-(U8-Pad5)
- R107 pad 2: Net-(R107-Pad2) -> Net-(U8-Pad12)
- R108 pad 2: Net-(R108-Pad2) -> Net-(U8-Pad3)
- R109 pad 2: Net-(R109-Pad2) -> Net-(U9-Pad5)
- R110 pad 2: Net-(R110-Pad2) -> Net-(U9-Pad12)
- R111 pad 2: Net-(R111-Pad2) -> Net-(U9-Pad10)
- R113 pad 2: Net-(R113-Pad2) -> Net-(U7-Pad10)
- R118 pad 1: Net-(R118-Pad1) -> Net-(R39-Pad2)
- R118 pad 2: Net-(R102-Pad2) -> Net-(U7-Pad5)
- R119 pad 2: Net-(R103-Pad2) -> Net-(U7-Pad12)
- R120 pad 1: Net-(R120-Pad1) -> Net-(R38-Pad2)
- R121 pad 2: Net-(R105-Pad2) -> Net-(U8-Pad5)
- R123 pad 2: Net-(R107-Pad2) -> Net-(U8-Pad12)
- R124 pad 2: Net-(R108-Pad2) -> Net-(U8-Pad3)
- R125 pad 1: Net-(R125-Pad1) -> Net-(R47-Pad2)
- R125 pad 2: Net-(R109-Pad2) -> Net-(U9-Pad5)
- R126 pad 2: Net-(R110-Pad2) -> Net-(U9-Pad12)
- R127 pad 2: Net-(R111-Pad2) -> Net-(U9-Pad10)
- R129 pad 2: Net-(R113-Pad2) -> Net-(U7-Pad10)
- R25 pad 2: Net-(R25-Pad2) -> Net-(R71-Pad1)
- R31 pad 2: Net-(R31-Pad2) -> Net-(R78-Pad1)
- R35 pad 2: Net-(R115-Pad1) -> Net-(R117-Pad1)
- R37 pad 2: Net-(R117-Pad1) -> Net-(R115-Pad1)
- R38 pad 2: Net-(R118-Pad1) -> Net-(R38-Pad2)
- R39 pad 2: Net-(R129-Pad1) -> Net-(R39-Pad2)
- R41 pad 2: Net-(R120-Pad1) -> Net-(R129-Pad1)
- R42 pad 2: Net-(R121-Pad1) -> Net-(R124-Pad1)
- R43 pad 2: Net-(R122-Pad1) -> Net-(R121-Pad1)
- R45 pad 2: Net-(R124-Pad1) -> Net-(R122-Pad1)
- R46 pad 2: Net-(R125-Pad1) -> Net-(R128-Pad1)
- R47 pad 2: Net-(R126-Pad1) -> Net-(R47-Pad2)
- R48 pad 2: Net-(R127-Pad1) -> Net-(R126-Pad1)
- R49 pad 2: Net-(R128-Pad1) -> Net-(R127-Pad1)
- R67 pad 1: Net-(R18-Pad2) -> Net-(R21-Pad2)
- R68 pad 2: Net-(R68-Pad2) -> Net-(U13-Pad3)
- R69 pad 1: Net-(R20-Pad2) -> Net-(R18-Pad2)
- R70 pad 1: Net-(R21-Pad2) -> Net-(R20-Pad2)
- R70 pad 2: Net-(R70-Pad2) -> Net-(U13-Pad10)
- R71 pad 1: Net-(R22-Pad2) -> Net-(R71-Pad1)
- R72 pad 1: Net-(R24-Pad2) -> Net-(R22-Pad2)
- R73 pad 1: Net-(R25-Pad2) -> Net-(R24-Pad2)
- R74 pad 1: Net-(R26-Pad2) -> Net-(R29-Pad2)
- R75 pad 1: Net-(R27-Pad2) -> Net-(R28-Pad2)
- R76 pad 1: Net-(R28-Pad2) -> Net-(R26-Pad2)
- R77 pad 1: Net-(R29-Pad2) -> Net-(R27-Pad2)
- R78 pad 1: Net-(R30-Pad2) -> Net-(R78-Pad1)
- R79 pad 1: Net-(R31-Pad2) -> Net-(R30-Pad2)
- R84 pad 2: Net-(R68-Pad2) -> Net-(U13-Pad3)
- R86 pad 2: Net-(R70-Pad2) -> Net-(U13-Pad10)
- U10 pad 10: Net-(R115-Pad2) -> Net-(R80-Pad2)
- U10 pad 12: Net-(R114-Pad2) -> Net-(R81-Pad2)
- U10 pad 3: Net-(R101-Pad2) -> Net-(R78-Pad2)
- U10 pad 5: Net-(R100-Pad2) -> Net-(R79-Pad2)
- U11 pad 10: Net-(R113-Pad2) -> Net-(R75-Pad2)
- U11 pad 12: Net-(R102-Pad2) -> Net-(R74-Pad2)
- U11 pad 3: Net-(R104-Pad2) -> Net-(R77-Pad2)
- U11 pad 5: Net-(R103-Pad2) -> Net-(R76-Pad2)
- U12 pad 10: Net-(R106-Pad2) -> Net-(R73-Pad2)
- U12 pad 11: -5V -> unconnected-(U12-Pad11)
- U12 pad 12: Net-(R105-Pad2) -> Net-(R71-Pad2)
- U12 pad 3: Net-(R108-Pad2) -> Net-(R66-Pad2)
- U12 pad 5: Net-(R107-Pad2) -> Net-(R72-Pad2)
- U13 pad 10: Net-(R110-Pad2) -> Net-(U13-Pad10)
- U13 pad 12: Net-(R109-Pad2) -> Net-(R67-Pad2)
- U13 pad 3: Net-(R112-Pad2) -> Net-(U13-Pad3)
- U13 pad 5: Net-(R111-Pad2) -> Net-(R69-Pad2)
- U14 pad 7: Net-(R31-Pad2) -> Net-(R78-Pad1)
- U19 pad 14: Net-(R117-Pad1) -> Net-(R115-Pad1)
- U19 pad 7: Net-(R115-Pad1) -> Net-(R117-Pad1)
- U20 pad 1: Net-(R118-Pad1) -> Net-(R38-Pad2)
- U20 pad 14: Net-(R120-Pad1) -> Net-(R129-Pad1)
- U20 pad 7: Net-(R129-Pad1) -> Net-(R39-Pad2)
- U21 pad 1: Net-(R121-Pad1) -> Net-(R124-Pad1)
- U21 pad 14: Net-(R124-Pad1) -> Net-(R122-Pad1)
- U21 pad 7: Net-(R122-Pad1) -> Net-(R121-Pad1)
- U22 pad 1: Net-(R125-Pad1) -> Net-(R128-Pad1)
- U22 pad 14: Net-(R128-Pad1) -> Net-(R127-Pad1)
- U22 pad 7: Net-(R126-Pad1) -> Net-(R47-Pad2)
- U22 pad 8: Net-(R127-Pad1) -> Net-(R126-Pad1)
- U4 pad 14: Net-(R25-Pad2) -> Net-(R71-Pad1)
- U6 pad 10: Net-(R80-Pad2) -> Net-(R115-Pad2)
- U6 pad 12: Net-(R81-Pad2) -> Net-(R100-Pad2)
- U6 pad 3: Net-(R78-Pad2) -> Net-(R101-Pad2)
- U6 pad 5: Net-(R79-Pad2) -> Net-(R114-Pad2)
- U7 pad 10: Net-(R76-Pad2) -> Net-(U7-Pad10)
- U7 pad 12: Net-(R77-Pad2) -> Net-(U7-Pad12)
- U7 pad 3: Net-(R74-Pad2) -> Net-(R104-Pad2)
- U7 pad 5: Net-(R75-Pad2) -> Net-(U7-Pad5)
- U8 pad 10: Net-(R72-Pad2) -> Net-(R106-Pad2)
- U8 pad 11: unconnected-(U8-Pad11) -> -5V
- U8 pad 12: Net-(R73-Pad2) -> Net-(U8-Pad12)
- U8 pad 3: Net-(R71-Pad2) -> Net-(U8-Pad3)
- U8 pad 5: Net-(R66-Pad2) -> Net-(U8-Pad5)
- U9 pad 10: Net-(R69-Pad2) -> Net-(U9-Pad10)
- U9 pad 12: Net-(R70-Pad2) -> Net-(U9-Pad12)
- U9 pad 3: Net-(R67-Pad2) -> Net-(R112-Pad2)
- U9 pad 5: Net-(R68-Pad2) -> Net-(U9-Pad5)
Routing:
- net Net-(J4-Pad3): track 0.00 -> 30.1 mm
- net Net-(J4-Pad34): track 0.00 -> 29.7 mm
- net Net-(J4-Pad6): track 0.00 -> 27.0 mm
- net Net-(J4-Pad31): track 0.00 -> 26.5 mm
- net Net-(J4-Pad7): track 0.00 -> 25.6 mm
- net Net-(J4-Pad30): track 0.00 -> 24.0 mm
- net Net-(J4-Pad10): track 0.00 -> 22.8 mm
- net Net-(J4-Pad11): track 0.00 -> 22.7 mm
- net Net-(J4-Pad27): track 0.00 -> 22.5 mm
- net Net-(J4-Pad33): track 0.00 -> 21.7 mm
- net Net-(J4-Pad4): track 0.00 -> 21.2 mm
- net Net-(J4-Pad26): track 0.00 -> 20.9 mm
- net Net-(J4-Pad14): track 0.00 -> 20.2 mm
- net Net-(J4-Pad22): track 0.00 -> 20.2 mm
- net Net-(J4-Pad15): track 0.00 -> 20.0 mm
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
Commit message: board2 progress
Parts:
- moved R65 29.3 mm to (170.2, 79.1), turned to 90 degrees
- moved R14 29.3 mm to (137.8, 79.1), turned to 90 degrees
- moved R15 29.0 mm to (137.8, 82.6), turned to -90 degrees
- moved R64 28.9 mm to (170.2, 82.6), turned to -90 degrees
- moved R49 28.6 mm to (168.1, 78.1)
- moved R30 28.6 mm to (139.8, 78.1)
- moved U22 28.4 mm to (163.2, 80.8)
- moved R33 28.4 mm to (149.5, 78.1)
- moved U14 28.4 mm to (144.5, 80.9)
- moved R46 28.3 mm to (158.4, 78.1)
- moved R48 28.3 mm to (168.1, 83.6)
- moved R47 28.3 mm to (158.4, 83.6)
- moved R31 28.2 mm to (139.7, 83.6)
- moved R32 28.2 mm to (149.4, 83.6)
- moved R1 27.9 mm to (151.8, 79.1), turned to 90 degrees
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Connections:
- J4 pad 11: Net-(J4-Pad11) -> Net-(U8-Pad8)
- J4 pad 12: Net-(J4-Pad12) -> Net-(U8-Pad13)
- J4 pad 13: Net-(J4-Pad13) -> Net-(U8-Pad1)
- J4 pad 14: Net-(J4-Pad14) -> Net-(U8-Pad6)
- J4 pad 15: Net-(J4-Pad15) -> Net-(U9-Pad8)
- J4 pad 16: Net-(J4-Pad16) -> Net-(U9-Pad13)
- J4 pad 17: Net-(J4-Pad17) -> Net-(U9-Pad1)
- J4 pad 18: Net-(J4-Pad18) -> Net-(U9-Pad6)
- J4 pad 19: Net-(J4-Pad19) -> Net-(U10-Pad8)
- J4 pad 20: Net-(J4-Pad20) -> Net-(U10-Pad13)
- J4 pad 21: Net-(J4-Pad21) -> Net-(U10-Pad1)
- J4 pad 22: Net-(J4-Pad22) -> Net-(U10-Pad6)
- J4 pad 23: Net-(J4-Pad23) -> Net-(U11-Pad8)
- J4 pad 24: Net-(J4-Pad24) -> Net-(U11-Pad13)
- J4 pad 25: Net-(J4-Pad25) -> Net-(U11-Pad1)
- J4 pad 26: Net-(J4-Pad26) -> Net-(U11-Pad6)
- J4 pad 27: Net-(J4-Pad27) -> Net-(U12-Pad8)
- J4 pad 28: Net-(J4-Pad28) -> Net-(U12-Pad13)
- J4 pad 29: Net-(J4-Pad29) -> Net-(U12-Pad1)
- J4 pad 30: Net-(J4-Pad30) -> Net-(U12-Pad6)
- J4 pad 31: Net-(J4-Pad31) -> Net-(U13-Pad8)
- J4 pad 32: Net-(J4-Pad32) -> Net-(U13-Pad13)
- J4 pad 33: Net-(J4-Pad33) -> Net-(U13-Pad1)
- J4 pad 34: Net-(J4-Pad34) -> Net-(U13-Pad6)
- R102 pad 2: Net-(U7-Pad5) -> Net-(R102-Pad2)
- R103 pad 2: Net-(U7-Pad12) -> Net-(R103-Pad2)
- R105 pad 2: Net-(U8-Pad5) -> Net-(R105-Pad2)
- R107 pad 2: Net-(U8-Pad12) -> Net-(U8-Pad10)
- R108 pad 2: Net-(U8-Pad3) -> Net-(R108-Pad2)
- R109 pad 2: Net-(U9-Pad5) -> Net-(R109-Pad2)
- R110 pad 2: Net-(U9-Pad12) -> Net-(U9-Pad10)
- R111 pad 2: Net-(U9-Pad10) -> Net-(U9-Pad12)
- R113 pad 2: Net-(U7-Pad10) -> Net-(R113-Pad2)
- R118 pad 2: Net-(U7-Pad5) -> Net-(R102-Pad2)
- R119 pad 2: Net-(U7-Pad12) -> Net-(R103-Pad2)
- R121 pad 2: Net-(U8-Pad5) -> Net-(R105-Pad2)
- R123 pad 2: Net-(U8-Pad12) -> Net-(U8-Pad10)
- R124 pad 2: Net-(U8-Pad3) -> Net-(R108-Pad2)
- R125 pad 2: Net-(U9-Pad5) -> Net-(R109-Pad2)
- R126 pad 2: Net-(U9-Pad12) -> Net-(U9-Pad10)
- R127 pad 2: Net-(U9-Pad10) -> Net-(U9-Pad12)
- R129 pad 2: Net-(U7-Pad10) -> Net-(R113-Pad2)
- R67 pad 2: Net-(R67-Pad2) -> Net-(U13-Pad10)
- R68 pad 2: Net-(U13-Pad3) -> Net-(U13-Pad5)
- R69 pad 2: Net-(R69-Pad2) -> Net-(U13-Pad3)
- R70 pad 2: Net-(U13-Pad10) -> Net-(U13-Pad12)
- R71 pad 2: Net-(R71-Pad2) -> Net-(U12-Pad10)
- R78 pad 2: Net-(R78-Pad2) -> Net-(U10-Pad5)
- R79 pad 2: Net-(R79-Pad2) -> Net-(U10-Pad3)
- R83 pad 2: Net-(R67-Pad2) -> Net-(U13-Pad10)
- R84 pad 2: Net-(U13-Pad3) -> Net-(U13-Pad5)
- R85 pad 2: Net-(R69-Pad2) -> Net-(U13-Pad3)
- R86 pad 2: Net-(U13-Pad10) -> Net-(U13-Pad12)
- R87 pad 2: Net-(R71-Pad2) -> Net-(U12-Pad10)
- R94 pad 2: Net-(R78-Pad2) -> Net-(U10-Pad5)
- R95 pad 2: Net-(R79-Pad2) -> Net-(U10-Pad3)
- U10 pad 1: Net-(J4-Pad22) -> Net-(U10-Pad1)
- U10 pad 10: Net-(R80-Pad2) -> Net-(R81-Pad2)
- U10 pad 12: Net-(R81-Pad2) -> Net-(R80-Pad2)
- U10 pad 13: Net-(J4-Pad19) -> Net-(U10-Pad13)
- U10 pad 14: Net-(J4-Pad19) -> Net-(U10-Pad13)
- U10 pad 2: Net-(J4-Pad22) -> Net-(U10-Pad1)
- U10 pad 3: Net-(R78-Pad2) -> Net-(U10-Pad3)
- U10 pad 5: Net-(R79-Pad2) -> Net-(U10-Pad5)
- U10 pad 6: Net-(J4-Pad21) -> Net-(U10-Pad6)
- U10 pad 7: Net-(J4-Pad21) -> Net-(U10-Pad6)
- U10 pad 8: Net-(J4-Pad20) -> Net-(U10-Pad8)
- U10 pad 9: Net-(J4-Pad20) -> Net-(U10-Pad8)
- U11 pad 1: Net-(J4-Pad26) -> Net-(U11-Pad1)
- U11 pad 10: Net-(R75-Pad2) -> Net-(R74-Pad2)
- U11 pad 12: Net-(R74-Pad2) -> Net-(R75-Pad2)
- U11 pad 13: Net-(J4-Pad23) -> Net-(U11-Pad13)
- U11 pad 14: Net-(J4-Pad23) -> Net-(U11-Pad13)
- U11 pad 2: Net-(J4-Pad26) -> Net-(U11-Pad1)
- U11 pad 3: Net-(R77-Pad2) -> Net-(R76-Pad2)
- U11 pad 5: Net-(R76-Pad2) -> Net-(R77-Pad2)
- U11 pad 6: Net-(J4-Pad25) -> Net-(U11-Pad6)
- U11 pad 7: Net-(J4-Pad25) -> Net-(U11-Pad6)
- U11 pad 8: Net-(J4-Pad24) -> Net-(U11-Pad8)
- U11 pad 9: Net-(J4-Pad24) -> Net-(U11-Pad8)
- U12 pad 1: Net-(J4-Pad30) -> Net-(U12-Pad1)
- U12 pad 10: Net-(R73-Pad2) -> Net-(U12-Pad10)
- U12 pad 11: unconnected-(U12-Pad11) -> -5V
- U12 pad 12: Net-(R71-Pad2) -> Net-(R73-Pad2)
- U12 pad 13: Net-(J4-Pad27) -> Net-(U12-Pad13)
- U12 pad 14: Net-(J4-Pad27) -> Net-(U12-Pad13)
- U12 pad 2: Net-(J4-Pad30) -> Net-(U12-Pad1)
- U12 pad 3: Net-(R66-Pad2) -> Net-(R72-Pad2)
- U12 pad 5: Net-(R72-Pad2) -> Net-(R66-Pad2)
- U12 pad 6: Net-(J4-Pad29) -> Net-(U12-Pad6)
- U12 pad 7: Net-(J4-Pad29) -> Net-(U12-Pad6)
- U12 pad 8: Net-(J4-Pad28) -> Net-(U12-Pad8)
- U12 pad 9: Net-(J4-Pad28) -> Net-(U12-Pad8)
- U13 pad 1: Net-(J4-Pad34) -> Net-(U13-Pad1)
- U13 pad 12: Net-(R67-Pad2) -> Net-(U13-Pad12)
- U13 pad 13: Net-(J4-Pad31) -> Net-(U13-Pad13)
- U13 pad 14: Net-(J4-Pad31) -> Net-(U13-Pad13)
- U13 pad 2: Net-(J4-Pad34) -> Net-(U13-Pad1)
- U13 pad 5: Net-(R69-Pad2) -> Net-(U13-Pad5)
- U13 pad 6: Net-(J4-Pad33) -> Net-(U13-Pad6)
- U13 pad 7: Net-(J4-Pad33) -> Net-(U13-Pad6)
- U13 pad 8: Net-(J4-Pad32) -> Net-(U13-Pad8)
- U13 pad 9: Net-(J4-Pad32) -> Net-(U13-Pad8)
- U6 pad 1: Net-(J4-Pad6) -> Net-(J4-Pad5)
- U6 pad 10: Net-(R115-Pad2) -> Net-(R100-Pad2)
- U6 pad 12: Net-(R100-Pad2) -> Net-(R115-Pad2)
- U6 pad 13: Net-(J4-Pad3) -> Net-(J4-Pad4)
- U6 pad 14: Net-(J4-Pad3) -> Net-(J4-Pad4)
- U6 pad 2: Net-(J4-Pad6) -> Net-(J4-Pad5)
- U6 pad 3: Net-(R101-Pad2) -> Net-(R114-Pad2)
- U6 pad 5: Net-(R114-Pad2) -> Net-(R101-Pad2)
- U6 pad 6: Net-(J4-Pad5) -> Net-(J4-Pad6)
- U6 pad 7: Net-(J4-Pad5) -> Net-(J4-Pad6)
- U6 pad 8: Net-(J4-Pad4) -> Net-(J4-Pad3)
- U6 pad 9: Net-(J4-Pad4) -> Net-(J4-Pad3)
- U7 pad 1: Net-(J4-Pad10) -> Net-(J4-Pad9)
- U7 pad 10: Net-(U7-Pad10) -> Net-(R103-Pad2)
- U7 pad 12: Net-(U7-Pad12) -> Net-(R113-Pad2)
- U7 pad 13: Net-(J4-Pad7) -> Net-(J4-Pad8)
- U7 pad 14: Net-(J4-Pad7) -> Net-(J4-Pad8)
- U7 pad 2: Net-(J4-Pad10) -> Net-(J4-Pad9)
- U7 pad 3: Net-(R104-Pad2) -> Net-(R102-Pad2)
- U7 pad 5: Net-(U7-Pad5) -> Net-(R104-Pad2)
- U7 pad 6: Net-(J4-Pad9) -> Net-(J4-Pad10)
- U7 pad 7: Net-(J4-Pad9) -> Net-(J4-Pad10)
- U7 pad 8: Net-(J4-Pad8) -> Net-(J4-Pad7)
- U7 pad 9: Net-(J4-Pad8) -> Net-(J4-Pad7)
- U8 pad 1: Net-(J4-Pad14) -> Net-(U8-Pad1)
- U8 pad 10: Net-(R106-Pad2) -> Net-(U8-Pad10)
- U8 pad 12: Net-(U8-Pad12) -> Net-(R106-Pad2)
- U8 pad 13: Net-(J4-Pad11) -> Net-(U8-Pad13)
- U8 pad 14: Net-(J4-Pad11) -> Net-(U8-Pad13)
- U8 pad 2: Net-(J4-Pad14) -> Net-(U8-Pad1)
- U8 pad 3: Net-(U8-Pad3) -> Net-(R105-Pad2)
- U8 pad 5: Net-(U8-Pad5) -> Net-(R108-Pad2)
- U8 pad 6: Net-(J4-Pad13) -> Net-(U8-Pad6)
- U8 pad 7: Net-(J4-Pad13) -> Net-(U8-Pad6)
- U8 pad 8: Net-(J4-Pad12) -> Net-(U8-Pad8)
- U8 pad 9: Net-(J4-Pad12) -> Net-(U8-Pad8)
- U9 pad 1: Net-(J4-Pad18) -> Net-(U9-Pad1)
- U9 pad 13: Net-(J4-Pad15) -> Net-(U9-Pad13)
- U9 pad 14: Net-(J4-Pad15) -> Net-(U9-Pad13)
- U9 pad 2: Net-(J4-Pad18) -> Net-(U9-Pad1)
- U9 pad 3: Net-(R112-Pad2) -> Net-(R109-Pad2)
- U9 pad 5: Net-(U9-Pad5) -> Net-(R112-Pad2)
- U9 pad 6: Net-(J4-Pad17) -> Net-(U9-Pad6)
- U9 pad 7: Net-(J4-Pad17) -> Net-(U9-Pad6)
- U9 pad 8: Net-(J4-Pad16) -> Net-(U9-Pad8)
- U9 pad 9: Net-(J4-Pad16) -> Net-(U9-Pad8)
Routing:
- net +5V: track 0.00 -> 109.6 mm, vias 0 -> 16
- net -5V: track 11.0 -> 97.6 mm, vias 0 -> 16
- net Net-(J4-Pad34): track 29.7 -> 0.00 mm
- net Net-(R101-Pad2): track 0.00 -> 29.3 mm
- net Net-(U13-Pad5): track 0.00 -> 28.8 mm
- net Net-(U13-Pad10): track 0.00 -> 28.5 mm
- net Net-(R114-Pad2): track 0.00 -> 28.4 mm
- net Net-(R100-Pad2): track 0.00 -> 28.3 mm
- net +2V5: track 0.00 -> 26.8 mm, vias 0 -> 16
- net Net-(U13-Pad12): track 0.00 -> 26.7 mm
- net Net-(J4-Pad31): track 26.5 -> 0.00 mm
- net Net-(R103-Pad2): track 0.00 -> 26.3 mm
- net Net-(J4-Pad3): track 30.1 -> 4.74 mm
- net Net-(R66-Pad2): track 0.00 -> 25.3 mm
- net Net-(R102-Pad2): track 0.00 -> 24.3 mm
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