File: KiCad/TheBoard_2/TheBoard_2.kicad_sch (KiCad schematic)
At the start: 163 parts, among them J1 Conn_01x03_Female, J2 Conn_01x03_Female, J3 Conn_01x16_Female, J4 Conn_01x36_Male, J5 Conn_01x16_Female, J6 Conn_01x02_Male, U1 MAX680CSA+T, U10 MCP6074-E/SL, U11 MCP6074-E/SL, U12 MCP6074-E/SL, U13 MCP6074-E/SL, U14 LM2902, U19 LM2902, U2 LM337_TO220, U20 LM2902, U21 LM2902, U22 LM2902, U3 LM2902, U4 LM2902, U5 LM2902, U6 MCP6074-E/SL, U7 MCP6074-E/SL, U8 MCP6074-E/SL, U9 MCP6074-E/SL

Commit message: board2 progress
Parts:
- J4: footprint Connector_PinHeader_2.54mm:PinHeader_2x18_P2.54mm_Horizontal -> Connector_PinHeader_2.54mm:PinHeader_1x36_P2.54mm_Horizontal
- renumbered U6 to U10, U7 to U11, U8 to U12, U9 to U13, U10 to U6, U11 to U7, U12 to U8, U13 to U9
Connections:
- net at R46.2, U22.1: now also R128.1; no longer R125.1
- net at R109.2, R125.2: now also U9.5 (VINB+); no longer U9.12 (VIND+)
- net at R26.2, U5.1: now also R76.1; no longer R74.1
- net at R28.2, U5.8: now also R75.1; no longer R76.1
- net at R30.2, U14.1: now also R79.1; no longer R78.1
- net at R42.2, U21.1: now also R124.1; no longer R121.1
- net at R72.2, R88.2: now also U12.5 (VINB+); no longer U12.10 (VINC+)
- net at R18.2, U3.1: now also R69.1; no longer R67.1
- net at R67.2, R83.2: now also U13.12 (VIND+); no longer U13.3 (VINA+)
- net at R100.2, R116.2: now also U6.12 (VIND+); no longer U6.5 (VINB+)
- net at R66.2, R82.2: now also U12.3 (VINA+); no longer U12.5 (VINB+)
- net at R31.2, U14.7: now also R78.1; no longer R79.1
- net at R45.2, U21.14: now also R122.1; no longer R124.1
- net at R49.2, U22.14: now also R127.1; no longer R128.1
- net at R27.2, U5.7: now also R77.1; no longer R75.1
- net at R75.2, R91.2: now also U11.10 (VINC+); no longer U11.5 (VINB+)
- net at R103.2, R119.2: now also U7.12 (VIND+); no longer U7.5 (VINB+)
- net at R105.2, R121.2: now also U8.5 (VINB+); no longer U8.12 (VIND+)
- net at R107.2, R123.2: now also U8.12 (VIND+); no longer U8.5 (VINB+)
- net at R41.2, U20.14: now also R129.1; no longer R120.1
- net at R102.2, R118.2: now also U7.5 (VINB+); no longer U7.12 (VIND+)
- net at R37.2, U19.14: now also R115.1; no longer R117.1
- net at R68.2, R84.2: now also U13.3 (VINA+); no longer U13.5 (VINB+)
- net at R20.2, U3.8: now also R70.1; no longer R69.1
- net at R47.2, U22.7: now also R125.1; no longer R126.1
- net at R114.2, R98.2: now also U6.5 (VINB+); no longer U6.12 (VIND+)
- net at R76.2, R92.2: now also U11.5 (VINB+); no longer U11.10 (VINC+)
- net at R35.2, U19.7: now also R117.1; no longer R115.1
- net at R39.2, U20.7: now also R118.1; no longer R129.1
- net at R29.2, U5.14: now also R74.1; no longer R77.1
- net at U9.1 (VOUTA), U9.2 (VINA-): now also J4.18 (Pin_18); no longer J4.34 (Pin_34)
- net at R110.2, R126.2: now also U9.12 (VIND+); no longer U9.10 (VINC+)
- net at U9.13 (VIND-), U9.14 (VOUTD): now also J4.15 (Pin_15); no longer J4.31 (Pin_31)
- net at R111.2, R127.2: now also U9.10 (VINC+); no longer U9.5 (VINB+)
- net at U9.6 (VINB-), U9.7 (VOUTB): now also J4.17 (Pin_17); no longer J4.33 (Pin_33)
- net at U9.8 (VOUTC), U9.9 (VINC-): now also J4.16 (Pin_16); no longer J4.32 (Pin_32)
- net at R43.2, U21.7: now also R121.1; no longer R122.1
- net at R77.2, R93.2: now also U11.3 (VINA+); no longer U11.12 (VIND+)
- net at R38.2, U20.1: now also R120.1; no longer R118.1
- net at U13.1 (VOUTA), U13.2 (VINA-): now also J4.34 (Pin_34); no longer J4.18 (Pin_18)
- net at R69.2, R85.2: now also U13.5 (VINB+); no longer U13.10 (VINC+)
- net at R70.2, R86.2: now also U13.10 (VINC+); no longer U13.12 (VIND+)
- net at U13.13 (VIND-), U13.14 (VOUTD): now also J4.31 (Pin_31); no longer J4.15 (Pin_15)
- net at U13.6 (VINB-), U13.7 (VOUTB): now also J4.33 (Pin_33); no longer J4.17 (Pin_17)
- net at U13.8 (VOUTC), U13.9 (VINC-): now also J4.32 (Pin_32); no longer J4.16 (Pin_16)
- net at R74.2, R90.2: now also U11.12 (VIND+); no longer U11.3 (VINA+)
- net at R22.2, U4.1: now also R72.1; no longer R71.1
- net at U6.1 (VOUTA), U6.2 (VINA-): now also J4.6 (Pin_6); no longer J4.22 (Pin_22)
- net at U6.13 (VIND-), U6.14 (VOUTD): now also J4.3 (Pin_3); no longer J4.19 (Pin_19)
- net at U6.6 (VINB-), U6.7 (VOUTB): now also J4.5 (Pin_5); no longer J4.21 (Pin_21)
- net at U6.8 (VOUTC), U6.9 (VINC-): now also J4.4 (Pin_4); no longer J4.20 (Pin_20)
- net at U11.1 (VOUTA), U11.2 (VINA-): now also J4.26 (Pin_26); no longer J4.10 (Pin_10)
- net at U12.13 (VIND-), U12.14 (VOUTD): now also J4.27 (Pin_27); no longer J4.11 (Pin_11)
- net at U12.8 (VOUTC), U12.9 (VINC-): now also J4.28 (Pin_28); no longer J4.12 (Pin_12)
- net at U12.6 (VINB-), U12.7 (VOUTB): now also J4.29 (Pin_29); no longer J4.13 (Pin_13)
- net at U12.1 (VOUTA), U12.2 (VINA-): now also J4.30 (Pin_30); no longer J4.14 (Pin_14)
- net at U7.13 (VIND-), U7.14 (VOUTD): now also J4.7 (Pin_7); no longer J4.23 (Pin_23)
- net at U7.8 (VOUTC), U7.9 (VINC-): now also J4.8 (Pin_8); no longer J4.24 (Pin_24)
- net at U7.6 (VINB-), U7.7 (VOUTB): now also J4.9 (Pin_9); no longer J4.25 (Pin_25)
- net at U7.1 (VOUTA), U7.2 (VINA-): now also J4.10 (Pin_10); no longer J4.26 (Pin_26)
- net at U8.13 (VIND-), U8.14 (VOUTD): now also J4.11 (Pin_11); no longer J4.27 (Pin_27)
- net at U8.8 (VOUTC), U8.9 (VINC-): now also J4.12 (Pin_12); no longer J4.28 (Pin_28)
- net at U8.6 (VINB-), U8.7 (VOUTB): now also J4.13 (Pin_13); no longer J4.29 (Pin_29)
- net at U10.13 (VIND-), U10.14 (VOUTD): now also J4.19 (Pin_19); no longer J4.3 (Pin_3)
- net at U8.1 (VOUTA), U8.2 (VINA-): now also J4.14 (Pin_14); no longer J4.30 (Pin_30)
- net at U10.8 (VOUTC), U10.9 (VINC-): now also J4.20 (Pin_20); no longer J4.4 (Pin_4)
- net at U10.6 (VINB-), U10.7 (VOUTB): now also J4.21 (Pin_21); no longer J4.5 (Pin_5)
- net at U10.1 (VOUTA), U10.2 (VINA-): now also J4.22 (Pin_22); no longer J4.6 (Pin_6)
- net at U11.13 (VIND-), U11.14 (VOUTD): now also J4.23 (Pin_23); no longer J4.7 (Pin_7)
- net at U11.8 (VOUTC), U11.9 (VINC-): now also J4.24 (Pin_24); no longer J4.8 (Pin_8)
- net at U11.6 (VINB-), U11.7 (VOUTB): now also J4.25 (Pin_25); no longer J4.9 (Pin_9)
- net at R24.2, U4.8: now also R73.1; no longer R72.1
- net at R48.2, U22.8: now also R126.1; no longer R127.1
- net at R21.2, U3.14: now also R67.1; no longer R70.1
- net at R25.2, U4.14: now also R71.1; no longer R73.1
- net at R73.2, R89.2: now also U12.10 (VINC+); no longer U12.12 (VIND+)
- net at R71.2, R87.2: now also U12.12 (VIND+); no longer U12.3 (VINA+)
Other:
- moved on the sheet: J4, R100, R101, R102, R103, R104, R105, R106, R107, R108, R109, R110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

Commit message: board2 progress
Connections:
- net -5V: now also U12.11 (VSS)
- net at R109.2, R125.2: now also U9.3 (VINA+); no longer U9.5 (VINB+)
- net at R72.2, R88.2: now also U12.3 (VINA+); no longer U12.5 (VINB+)
- net at R67.2, R83.2: now also U13.10 (VINC+); no longer U13.12 (VIND+)
- net at R100.2, R116.2: now also U6.10 (VINC+); no longer U6.12 (VIND+)
- net at R66.2, R82.2: now also U12.5 (VINB+); no longer U12.3 (VINA+)
- net at R80.2, R96.2: now also U10.12 (VIND+); no longer U10.10 (VINC+)
- net at R75.2, R91.2: now also U11.12 (VIND+); no longer U11.10 (VINC+)
- net at R103.2, R119.2: now also U7.10 (VINC+); no longer U7.12 (VIND+)
- net at R105.2, R121.2: now also U8.3 (VINA+); no longer U8.5 (VINB+)
- net at R79.2, R95.2: now also U10.3 (VINA+); no longer U10.5 (VINB+)
- net at R107.2, R123.2: now also U8.10 (VINC+); no longer U8.12 (VIND+)
- net at R104.2, R120.2: now also U7.5 (VINB+); no longer U7.3 (VINA+)
- net at R102.2, R118.2: now also U7.3 (VINA+); no longer U7.5 (VINB+)
- net at R68.2, R84.2: now also U13.5 (VINB+); no longer U13.3 (VINA+)
- net at R114.2, R98.2: now also U6.3 (VINA+); no longer U6.5 (VINB+)
- net at R76.2, R92.2: now also U11.3 (VINA+); no longer U11.5 (VINB+)
- net at R115.2, R99.2: now also U6.12 (VIND+); no longer U6.10 (VINC+)
- net at R113.2, R129.2: now also U7.12 (VIND+); no longer U7.10 (VINC+)
- net at U9.1 (VOUTA), U9.2 (VINA-): now also J4.17 (Pin_17); no longer J4.18 (Pin_18)
- net at R111.2, R127.2: now also U9.12 (VIND+); no longer U9.10 (VINC+)
- net at R110.2, R126.2: now also U9.10 (VINC+); no longer U9.12 (VIND+)
- net at U9.13 (VIND-), U9.14 (VOUTD): now also J4.16 (Pin_16); no longer J4.15 (Pin_15)
- net at R112.2, R128.2: now also U9.5 (VINB+); no longer U9.3 (VINA+)
- net at U9.6 (VINB-), U9.7 (VOUTB): now also J4.18 (Pin_18); no longer J4.17 (Pin_17)
- net at U9.8 (VOUTC), U9.9 (VINC-): now also J4.15 (Pin_15); no longer J4.16 (Pin_16)
- net at R77.2, R93.2: now also U11.5 (VINB+); no longer U11.3 (VINA+)
- net at U13.1 (VOUTA), U13.2 (VINA-): now also J4.33 (Pin_33); no longer J4.34 (Pin_34)
- net at R70.2, R86.2: now also U13.12 (VIND+); no longer U13.10 (VINC+)
- net at U13.13 (VIND-), U13.14 (VOUTD): now also J4.32 (Pin_32); no longer J4.31 (Pin_31)
- net at R69.2, R85.2: now also U13.3 (VINA+); no longer U13.5 (VINB+)
- net at U13.6 (VINB-), U13.7 (VOUTB): now also J4.34 (Pin_34); no longer J4.33 (Pin_33)
- net at U13.8 (VOUTC), U13.9 (VINC-): now also J4.31 (Pin_31); no longer J4.32 (Pin_32)
- net at R74.2, R90.2: now also U11.10 (VINC+); no longer U11.12 (VIND+)
- net at R106.2, R122.2: now also U8.12 (VIND+); no longer U8.10 (VINC+)
- net at U6.1 (VOUTA), U6.2 (VINA-): now also J4.5 (Pin_5); no longer J4.6 (Pin_6)
- net at U6.13 (VIND-), U6.14 (VOUTD): now also J4.4 (Pin_4); no longer J4.3 (Pin_3)
- net at R101.2, R117.2: now also U6.5 (VINB+); no longer U6.3 (VINA+)
- net at U6.6 (VINB-), U6.7 (VOUTB): now also J4.6 (Pin_6); no longer J4.5 (Pin_5)
- net at U6.8 (VOUTC), U6.9 (VINC-): now also J4.3 (Pin_3); no longer J4.4 (Pin_4)
- net at U7.1 (VOUTA), U7.2 (VINA-): now also J4.9 (Pin_9); no longer J4.10 (Pin_10)
- net at U8.13 (VIND-), U8.14 (VOUTD): now also J4.12 (Pin_12); no longer J4.11 (Pin_11)
- net at U8.8 (VOUTC), U8.9 (VINC-): now also J4.11 (Pin_11); no longer J4.12 (Pin_12)
- net at U8.6 (VINB-), U8.7 (VOUTB): now also J4.14 (Pin_14); no longer J4.13 (Pin_13)
- net at U8.1 (VOUTA), U8.2 (VINA-): now also J4.13 (Pin_13); no longer J4.14 (Pin_14)
- net at U10.13 (VIND-), U10.14 (VOUTD): now also J4.20 (Pin_20); no longer J4.19 (Pin_19)
- net at U10.8 (VOUTC), U10.9 (VINC-): now also J4.19 (Pin_19); no longer J4.20 (Pin_20)
- net at U10.6 (VINB-), U10.7 (VOUTB): now also J4.22 (Pin_22); no longer J4.21 (Pin_21)
- net at U10.1 (VOUTA), U10.2 (VINA-): now also J4.21 (Pin_21); no longer J4.22 (Pin_22)
- net at U11.13 (VIND-), U11.14 (VOUTD): now also J4.24 (Pin_24); no longer J4.23 (Pin_23)
- net at U11.8 (VOUTC), U11.9 (VINC-): now also J4.23 (Pin_23); no longer J4.24 (Pin_24)
- net at U11.6 (VINB-), U11.7 (VOUTB): now also J4.26 (Pin_26); no longer J4.25 (Pin_25)
- net at U11.1 (VOUTA), U11.2 (VINA-): now also J4.25 (Pin_25); no longer J4.26 (Pin_26)
- net at U12.13 (VIND-), U12.14 (VOUTD): now also J4.28 (Pin_28); no longer J4.27 (Pin_27)
- net at U12.8 (VOUTC), U12.9 (VINC-): now also J4.27 (Pin_27); no longer J4.28 (Pin_28)
- net at U12.6 (VINB-), U12.7 (VOUTB): now also J4.30 (Pin_30); no longer J4.29 (Pin_29)
- net at U12.1 (VOUTA), U12.2 (VINA-): now also J4.29 (Pin_29); no longer J4.30 (Pin_30)
- net at U7.13 (VIND-), U7.14 (VOUTD): now also J4.8 (Pin_8); no longer J4.7 (Pin_7)
- net at U7.8 (VOUTC), U7.9 (VINC-): now also J4.7 (Pin_7); no longer J4.8 (Pin_8)
- net at U7.6 (VINB-), U7.7 (VOUTB): now also J4.10 (Pin_10); no longer J4.9 (Pin_9)
- net at R108.2, R124.2: now also U8.5 (VINB+); no longer U8.3 (VINA+)
- net at R73.2, R89.2: now also U12.12 (VIND+); no longer U12.10 (VINC+)
- net at R81.2, R97.2: now also U10.10 (VINC+); no longer U10.12 (VIND+)
- net at R78.2, R94.2: now also U10.5 (VINB+); no longer U10.3 (VINA+)
- net at R71.2, R87.2: now also U12.10 (VINC+); no longer U12.12 (VIND+)
